Commit message: initial commit

File: mcorin_description/urdfs/common.xacro (robot description, xacro)
@@ -3,7 +3,7 @@
 	<xacro:property name="PI" value="3.1415926535897931"/>
 	<!-- standard distances -->
-	<xacro:property name="trunk_x" value="0.35"/> 		<!-- distance between front & back  joints -->
-	<xacro:property name="trunk_y" value="0.15"/> 		<!-- distance between left  & right joints -->
-	<xacro:property name="trunk_z" value="0.04"/>
+	<xacro:property name="trunk_x" value="0.1"/> 		<!-- distance between front & back  joints -->
+	<xacro:property name="trunk_y" value="0.1"/> 		<!-- distance between left  & right joints -->
+	<xacro:property name="trunk_z" value="0.1"/>
 	<!--  Joint parameters -->
 	<xacro:property name="MX64_damping"   value="0.15" /> 					<!-- real: 0.2 		-->
