Commit message: corIIn working with new dynamixel library, controllable via rosparam

File: mcorin_description/robots/fixed_mcorin.urdf (robot description, URDF)
Before this commit: robot corin, 27 links, 26 joints
Links:
- link lf_foot: mass 0.005 -> 0.04; geometry collision sphere radius=0.016; visual sphere radius=0.016
- link lf_hipassembly: mass 0.175 -> 0.0406; geometry collision mesh filename=package://mcorin_description/meshes/Coxa_collision.STL scale=1 1 1; visual mesh filename=package://mcorin_description/meshes/Coxa.STL scale=1 1 1
- link lf_lowerleg: mass 0.0537 -> 0.076; geometry collision mesh filename=package://mcorin_description/meshes/Tibia_collision.STL scale=1 1 1; visual mesh filename=package://mcorin_description/meshes/Tibia.STL scale=1 1 1
- link lf_upperleg: mass 0.1554 -> 0.35; geometry collision box size=0.15 0.04 0.04; visual mesh filename=package://mcorin_description/meshes/Femur.STL scale=1 1 1
- link lm_foot: mass 0.005 -> 0.04; geometry collision sphere radius=0.016; visual sphere radius=0.016
- link lm_hipassembly: mass 0.175 -> 0.0406; geometry collision mesh filename=package://mcorin_description/meshes/Coxa_collision.STL scale=1 1 1; visual mesh filename=package://mcorin_description/meshes/Coxa.STL scale=1 1 1
- link lm_lowerleg: mass 0.0537 -> 0.076; geometry collision mesh filename=package://mcorin_description/meshes/Tibia_collision.STL scale=1 1 1; visual mesh filename=package://mcorin_description/meshes/Tibia.STL scale=1 1 1
- link lm_upperleg: mass 0.1554 -> 0.35; geometry collision box size=0.15 0.04 0.04; visual mesh filename=package://mcorin_description/meshes/Femur.STL scale=1 1 1
- link lr_foot: mass 0.005 -> 0.04; geometry collision sphere radius=0.016; visual sphere radius=0.016
- link lr_hipassembly: mass 0.175 -> 0.0406; geometry collision mesh filename=package://mcorin_description/meshes/Coxa_collision.STL scale=1 1 1; visual mesh filename=package://mcorin_description/meshes/Coxa.STL scale=1 1 1
- link lr_lowerleg: mass 0.0537 -> 0.076; geometry collision mesh filename=package://mcorin_description/meshes/Tibia_collision.STL scale=1 1 1; visual mesh filename=package://mcorin_description/meshes/Tibia.STL scale=1 1 1
- link lr_upperleg: mass 0.1554 -> 0.35; geometry collision box size=0.15 0.04 0.04; visual mesh filename=package://mcorin_description/meshes/Femur.STL scale=1 1 1
- link rf_foot: mass 0.005 -> 0.04; geometry collision sphere radius=0.016; visual sphere radius=0.016
- link rf_hipassembly: mass 0.175 -> 0.0406; geometry collision mesh filename=package://mcorin_description/meshes/Coxa_collision.STL scale=1 1 1; visual mesh filename=package://mcorin_description/meshes/Coxa.STL scale=1 1 1
- link rf_lowerleg: mass 0.0537 -> 0.076; geometry collision mesh filename=package://mcorin_description/meshes/Tibia_collision.STL scale=1 1 1; visual mesh filename=package://mcorin_description/meshes/Tibia.STL scale=1 1 1
- link rf_upperleg: mass 0.1554 -> 0.35; geometry collision box size=0.15 0.04 0.04; visual mesh filename=package://mcorin_description/meshes/Femur.STL scale=1 1 1
- link rm_foot: mass 0.005 -> 0.04; geometry collision sphere radius=0.016; visual sphere radius=0.016
- link rm_hipassembly: mass 0.175 -> 0.0406; geometry collision mesh filename=package://mcorin_description/meshes/Coxa_collision.STL scale=1 1 1; visual mesh filename=package://mcorin_description/meshes/Coxa.STL scale=1 1 1
- link rm_lowerleg: mass 0.0537 -> 0.076; geometry collision mesh filename=package://mcorin_description/meshes/Tibia_collision.STL scale=1 1 1; visual mesh filename=package://mcorin_description/meshes/Tibia.STL scale=1 1 1
- link rm_upperleg: mass 0.1554 -> 0.35; geometry collision box size=0.15 0.04 0.04; visual mesh filename=package://mcorin_description/meshes/Femur.STL scale=1 1 1
- link rr_foot: mass 0.005 -> 0.04; geometry collision sphere radius=0.016; visual sphere radius=0.016
- link rr_hipassembly: mass 0.175 -> 0.0406; geometry collision mesh filename=package://mcorin_description/meshes/Coxa_collision.STL scale=1 1 1; visual mesh filename=package://mcorin_description/meshes/Coxa.STL scale=1 1 1
- link rr_lowerleg: mass 0.0537 -> 0.076; geometry collision mesh filename=package://mcorin_description/meshes/Tibia_collision.STL scale=1 1 1; visual mesh filename=package://mcorin_description/meshes/Tibia.STL scale=1 1 1
- link rr_upperleg: mass 0.1554 -> 0.35; geometry collision box size=0.15 0.04 0.04; visual mesh filename=package://mcorin_description/meshes/Femur.STL scale=1 1 1
- link trunk: mass 1.5 -> 1.58; geometry collision mesh filename=package://mcorin_description/meshes/Body_collision.STL scale=1 1 1; visual mesh filename=package://mcorin_description/meshes/Body.STL scale=1 1 1
Joints:
- joint lf_foot_joint: origin xyz=0.16 0 0 rpy=0 0 0 -> xyz=0.134 0 0 rpy=0 0 0
- joint lf_q1_joint: origin xyz=0.175 0.075 0 rpy=0 0 1.57079632679 -> xyz=0.115 0.09 0 rpy=0 0 0.872664625997
- joint lf_q2_joint: origin xyz=0.077 0 0 rpy=1.57079632679 0 0 -> xyz=0.06 0 0 rpy=1.57079632679 0 0
- joint lm_foot_joint: origin xyz=0.16 0 0 rpy=0 0 0 -> xyz=0.134 0 0 rpy=0 0 0
- joint lm_q1_joint: origin xyz=0 0.075 0 rpy=0 0 1.57079632679 -> xyz=0 0.09 0 rpy=0 0 1.57079632679
- joint lm_q2_joint: origin xyz=0.077 0 0 rpy=1.57079632679 0 0 -> xyz=0.06 0 0 rpy=1.57079632679 0 0
- joint lr_foot_joint: origin xyz=0.16 0 0 rpy=0 0 0 -> xyz=0.134 0 0 rpy=0 0 0
- joint lr_q1_joint: origin xyz=-0.175 0.075 0 rpy=0 0 1.57079632679 -> xyz=-0.115 0.09 0 rpy=0 0 2.26892802759
- joint lr_q2_joint: origin xyz=0.077 0 0 rpy=1.57079632679 0 0 -> xyz=0.06 0 0 rpy=1.57079632679 0 0
- joint rf_foot_joint: origin xyz=0.16 0 0 rpy=0 0 0 -> xyz=0.134 0 0 rpy=0 0 0
- joint rf_q1_joint: origin xyz=0.175 -0.075 0 rpy=0 0 -1.57079632679 -> xyz=0.115 -0.09 0 rpy=0 0 -0.872664625997
- joint rf_q2_joint: origin xyz=0.077 0 0 rpy=1.57079632679 0 0 -> xyz=0.06 0 0 rpy=1.57079632679 0 0
- joint rm_foot_joint: origin xyz=0.16 0 0 rpy=0 0 0 -> xyz=0.134 0 0 rpy=0 0 0
- joint rm_q1_joint: origin xyz=0 -0.075 0 rpy=0 0 -1.57079632679 -> xyz=0 -0.09 0 rpy=0 0 -1.57079632679
- joint rm_q2_joint: origin xyz=0.077 0 0 rpy=1.57079632679 0 0 -> xyz=0.06 0 0 rpy=1.57079632679 0 0
- joint rr_foot_joint: origin xyz=0.16 0 0 rpy=0 0 0 -> xyz=0.134 0 0 rpy=0 0 0
- joint rr_q1_joint: origin xyz=-0.175 -0.075 0 rpy=0 0 -1.57079632679 -> xyz=-0.115 -0.09 0 rpy=0 0 -2.26892802759
- joint rr_q2_joint: origin xyz=0.077 0 0 rpy=1.57079632679 0 0 -> xyz=0.06 0 0 rpy=1.57079632679 0 0

File: mcorin_description/robots/mCorin_fixed.urdf.xacro (robot description, xacro)
@@ -29,5 +29,5 @@
 		parent="trunk"
 		load_force_sensors="true">
-		<origin xyz="${trunk_x/2} ${trunk_y/2} 0" rpy="0 0 ${PI/2}"/>
+		<origin xyz="${trunk_x/2} ${trunk_y/2} 0" rpy="0 0 ${50*PI/180}"/>
 	</xacro:mCorin_leg>
 	<xacro:mCorin_leg
@@ -41,5 +41,5 @@
 		parent="trunk"
 		load_force_sensors="false">
-		<origin xyz="${-trunk_x/2} ${trunk_y/2} 0" rpy="0 0 ${PI/2}"/>
+		<origin xyz="${-trunk_x/2} ${trunk_y/2} 0" rpy="0 0 ${PI/2+40*PI/180}"/>
 	</xacro:mCorin_leg>
 	<xacro:mCorin_leg
@@ -47,5 +47,5 @@
 		parent="trunk"
 		load_force_sensors="true">
-		<origin xyz="${trunk_x/2} ${-trunk_y/2} 0" rpy="0 0 ${-PI/2}"/>
+		<origin xyz="${trunk_x/2} ${-trunk_y/2} 0" rpy="0 0 ${-50*PI/180}"/>
 	</xacro:mCorin_leg>
 	<xacro:mCorin_leg
@@ -59,5 +59,5 @@
 		parent="trunk"
 		load_force_sensors="false">
-		<origin xyz="${-trunk_x/2} ${-trunk_y/2} 0" rpy="0 0 ${-PI/2}"/>
+		<origin xyz="${-trunk_x/2} ${-trunk_y/2} 0" rpy="0 0 ${-PI/2-40*PI/180}"/>
 	</xacro:mCorin_leg>
 	<!-- Sensors -->

File: mcorin_description/robots/mCorin_model.urdf.xacro (robot description, xacro)
@@ -29,5 +29,5 @@
 		parent="trunk"
 		load_force_sensors="true">
-		<origin xyz="${trunk_x/2} ${trunk_y/2} 0" rpy="0 0 ${PI/2}"/>
+		<origin xyz="${trunk_x/2} ${trunk_y/2} 0" rpy="0 0 ${50*PI/180}"/>
 	</xacro:mCorin_leg>
 	<xacro:mCorin_leg
@@ -41,5 +41,5 @@
 		parent="trunk"
 		load_force_sensors="false">
-		<origin xyz="${-trunk_x/2} ${trunk_y/2} 0" rpy="0 0 ${PI/2}"/>
+		<origin xyz="${-trunk_x/2} ${trunk_y/2} 0" rpy="0 0 ${PI/2+40*PI/180}"/>
 	</xacro:mCorin_leg>
 	<xacro:mCorin_leg
@@ -47,5 +47,5 @@
 		parent="trunk"
 		load_force_sensors="true">
-		<origin xyz="${trunk_x/2} ${-trunk_y/2} 0" rpy="0 0 ${-PI/2}"/>
+		<origin xyz="${trunk_x/2} ${-trunk_y/2} 0" rpy="0 0 ${-50*PI/180}"/>
 	</xacro:mCorin_leg>
 	<xacro:mCorin_leg
@@ -59,5 +59,5 @@
 		parent="trunk"
 		load_force_sensors="false">
-		<origin xyz="${-trunk_x/2} ${-trunk_y/2} 0" rpy="0 0 ${-PI/2}"/>
+		<origin xyz="${-trunk_x/2} ${-trunk_y/2} 0" rpy="0 0 ${-PI/2-40*PI/180}"/>
 	</xacro:mCorin_leg>
 	<!-- Sensors -->
@@ -75,5 +75,5 @@
 		lidar_topic="lidar/data"
 		update_rate="100">
-		<origin xyz="0.06 0.0 0.03" rpy="0 0 ${PI/2}"/>
+		<origin xyz="0.06 0.0 0.04" rpy="0 0 ${PI/2}"/>
 	</xacro:LIDAR>
 </robot>

File: mcorin_description/robots/mcorin.urdf (robot description, URDF)
Before this commit: robot corin, 28 links, 27 joints
Links:
- link lf_foot: geometry collision sphere radius=0.016; visual sphere radius=0.016
- link lf_hipassembly: geometry collision mesh filename=package://mcorin_description/meshes/Coxa_collision.STL scale=1 1 1; visual mesh filename=package://mcorin_description/meshes/Coxa.STL scale=1 1 1
- link lf_lowerleg: geometry collision mesh filename=package://mcorin_description/meshes/Tibia_collision.STL scale=1 1 1; visual mesh filename=package://mcorin_description/meshes/Tibia.STL scale=1 1 1
- link lf_upperleg: geometry collision box size=0.15 0.04 0.04; visual mesh filename=package://mcorin_description/meshes/Femur.STL scale=1 1 1
- link lm_foot: geometry collision sphere radius=0.016; visual sphere radius=0.016
- link lm_hipassembly: geometry collision mesh filename=package://mcorin_description/meshes/Coxa_collision.STL scale=1 1 1; visual mesh filename=package://mcorin_description/meshes/Coxa.STL scale=1 1 1
- link lm_lowerleg: geometry collision mesh filename=package://mcorin_description/meshes/Tibia_collision.STL scale=1 1 1; visual mesh filename=package://mcorin_description/meshes/Tibia.STL scale=1 1 1
- link lm_upperleg: geometry collision box size=0.15 0.04 0.04; visual mesh filename=package://mcorin_description/meshes/Femur.STL scale=1 1 1
- link lr_foot: geometry collision sphere radius=0.016; visual sphere radius=0.016
- link lr_hipassembly: geometry collision mesh filename=package://mcorin_description/meshes/Coxa_collision.STL scale=1 1 1; visual mesh filename=package://mcorin_description/meshes/Coxa.STL scale=1 1 1
- link lr_lowerleg: geometry collision mesh filename=package://mcorin_description/meshes/Tibia_collision.STL scale=1 1 1; visual mesh filename=package://mcorin_description/meshes/Tibia.STL scale=1 1 1
- link lr_upperleg: geometry collision box size=0.15 0.04 0.04; visual mesh filename=package://mcorin_description/meshes/Femur.STL scale=1 1 1
- link rf_foot: geometry collision sphere radius=0.016; visual sphere radius=0.016
- link rf_hipassembly: geometry collision mesh filename=package://mcorin_description/meshes/Coxa_collision.STL scale=1 1 1; visual mesh filename=package://mcorin_description/meshes/Coxa.STL scale=1 1 1
- link rf_lowerleg: geometry collision mesh filename=package://mcorin_description/meshes/Tibia_collision.STL scale=1 1 1; visual mesh filename=package://mcorin_description/meshes/Tibia.STL scale=1 1 1
- link rf_upperleg: geometry collision box size=0.15 0.04 0.04; visual mesh filename=package://mcorin_description/meshes/Femur.STL scale=1 1 1
- link rm_foot: geometry collision sphere radius=0.016; visual sphere radius=0.016
- link rm_hipassembly: geometry collision mesh filename=package://mcorin_description/meshes/Coxa_collision.STL scale=1 1 1; visual mesh filename=package://mcorin_description/meshes/Coxa.STL scale=1 1 1
- link rm_lowerleg: geometry collision mesh filename=package://mcorin_description/meshes/Tibia_collision.STL scale=1 1 1; visual mesh filename=package://mcorin_description/meshes/Tibia.STL scale=1 1 1
- link rm_upperleg: geometry collision box size=0.15 0.04 0.04; visual mesh filename=package://mcorin_description/meshes/Femur.STL scale=1 1 1
- link rr_foot: geometry collision sphere radius=0.016; visual sphere radius=0.016
- link rr_hipassembly: geometry collision mesh filename=package://mcorin_description/meshes/Coxa_collision.STL scale=1 1 1; visual mesh filename=package://mcorin_description/meshes/Coxa.STL scale=1 1 1
- link rr_lowerleg: geometry collision mesh filename=package://mcorin_description/meshes/Tibia_collision.STL scale=1 1 1; visual mesh filename=package://mcorin_description/meshes/Tibia.STL scale=1 1 1
- link rr_upperleg: geometry collision box size=0.15 0.04 0.04; visual mesh filename=package://mcorin_description/meshes/Femur.STL scale=1 1 1
- link trunk: geometry collision mesh filename=package://mcorin_description/meshes/Body_collision.STL scale=1 1 1; visual mesh filename=package://mcorin_description/meshes/Body.STL scale=1 1 1
Joints:
- joint lf_foot_joint: origin xyz=0.16 0 0 rpy=0 0 0 -> xyz=0.134 0 0 rpy=0 0 0
- joint lf_q1_joint: origin xyz=0.175 0.075 0 rpy=0 0 1.57079632679 -> xyz=0.115 0.09 0 rpy=0 0 0.872664625997
- joint lf_q2_joint: origin xyz=0.077 0 0 rpy=1.57079632679 0 0 -> xyz=0.06 0 0 rpy=1.57079632679 0 0
- joint lm_foot_joint: origin xyz=0.16 0 0 rpy=0 0 0 -> xyz=0.134 0 0 rpy=0 0 0
- joint lm_q1_joint: origin xyz=0 0.075 0 rpy=0 0 1.57079632679 -> xyz=0 0.09 0 rpy=0 0 1.57079632679
- joint lm_q2_joint: origin xyz=0.077 0 0 rpy=1.57079632679 0 0 -> xyz=0.06 0 0 rpy=1.57079632679 0 0
- joint lr_foot_joint: origin xyz=0.16 0 0 rpy=0 0 0 -> xyz=0.134 0 0 rpy=0 0 0
- joint lr_q1_joint: origin xyz=-0.175 0.075 0 rpy=0 0 1.57079632679 -> xyz=-0.115 0.09 0 rpy=0 0 2.26892802759
- joint lr_q2_joint: origin xyz=0.077 0 0 rpy=1.57079632679 0 0 -> xyz=0.06 0 0 rpy=1.57079632679 0 0
- joint rf_foot_joint: origin xyz=0.16 0 0 rpy=0 0 0 -> xyz=0.134 0 0 rpy=0 0 0
- joint rf_q1_joint: origin xyz=0.175 -0.075 0 rpy=0 0 -1.57079632679 -> xyz=0.115 -0.09 0 rpy=0 0 -0.872664625997
- joint rf_q2_joint: origin xyz=0.077 0 0 rpy=1.57079632679 0 0 -> xyz=0.06 0 0 rpy=1.57079632679 0 0
- joint rm_foot_joint: origin xyz=0.16 0 0 rpy=0 0 0 -> xyz=0.134 0 0 rpy=0 0 0
- joint rm_q1_joint: origin xyz=0 -0.075 0 rpy=0 0 -1.57079632679 -> xyz=0 -0.09 0 rpy=0 0 -1.57079632679
- joint rm_q2_joint: origin xyz=0.077 0 0 rpy=1.57079632679 0 0 -> xyz=0.06 0 0 rpy=1.57079632679 0 0
- joint rr_foot_joint: origin xyz=0.16 0 0 rpy=0 0 0 -> xyz=0.134 0 0 rpy=0 0 0
- joint rr_q1_joint: origin xyz=-0.175 -0.075 0 rpy=0 0 -1.57079632679 -> xyz=-0.115 -0.09 0 rpy=0 0 -2.26892802759
- joint rr_q2_joint: origin xyz=0.077 0 0 rpy=1.57079632679 0 0 -> xyz=0.06 0 0 rpy=1.57079632679 0 0
- joint trunk_lidar_joint: origin xyz=0.06 0.0 0.03 rpy=0 0 1.57079632679 -> xyz=0.06 0.0 0.04 rpy=0 0 1.57079632679

File: mcorin_description/urdfs/common.xacro (robot description, xacro)
@@ -3,14 +3,15 @@
 	<xacro:property name="PI" value="3.1415926535897931"/>
 	<!-- standard distances -->
-	<xacro:property name="trunk_x" value="0.1"/> 		<!-- distance between front & back  joints -->
-	<xacro:property name="trunk_y" value="0.1"/> 		<!-- distance between left  & right joints -->
-	<xacro:property name="trunk_z" value="0.1"/>
+	<xacro:property name="trunk_x" value="0.23"/> 		<!-- distance between front & back  joints -->
+	<xacro:property name="trunk_y" value="0.18"/> 		<!-- distance between left  & right joints -->
+	<xacro:property name="trunk_z" value="0.07"/>
 	<!--  Joint parameters -->
 	<xacro:property name="MX64_damping"   value="0.15" /> 					<!-- real: 0.2 		-->
 	<xacro:property name="MX64_effort"    value="2.85" /> 					<!-- real: 2.85 Nm 	-->
 	<xacro:property name="MX64_velocity"  value="5.23" />
-	<xacro:property name="cox_joint_lim" value="1.6"  /> 		<!-- 90 deg "0.8726" -->
-	<xacro:property name="fem_joint_lim" value="2.36" />
-	<xacro:property name="tib_joint_lim" value="3.1" /> 	<!-- 2.62 -->
+	<xacro:property name="cox_joint_lim" value="1.00" />	<!-- 57deg -->
+	<xacro:property name="cxm_joint_lim" value="0.84" />	<!-- 48deg -->
+	<xacro:property name="fem_joint_lim" value="2.22" />	<!-- 127deg -->
+	<xacro:property name="tib_joint_lim" value="2.79" /> 	<!-- 160.5 -->
 	<!-- Inertial values -->
 	<!-- Trunk  -->
@@ -18,5 +19,5 @@
 	<xacro:property name="ycom_trunk" value="0.0"/>
 	<xacro:property name="zcom_trunk" value="0.0"/>
-	<xacro:property name="m_trunk" 	  value="1.50"/> <!-- initially 1.5 -->
+	<xacro:property name="m_trunk" 	  value="1.58"/> <!-- initially 1.5 -->
 	<xacro:property name="ixx_trunk"  value="${ (m_trunk/12)*(trunk_y*trunk_y + trunk_z*trunk_z) } "/>
 	<xacro:property name="iyy_trunk"  value="${ (m_trunk/12)*(trunk_x*trunk_x + trunk_z*trunk_z) } "/>
@@ -26,52 +27,52 @@
 	<xacro:property name="iyz_trunk"  value="0.0"/>
 	<!-- Coxa assembly -->
-	<xacro:property name="coxa_l"     value="0.077"  />
-	<xacro:property name="coxa_w"     value="0.046"  />
-	<xacro:property name="coxa_d"     value="0.0528" />
-	<xacro:property name="coxa_cl"    value="0.0611" />
-	<xacro:property name="coxa_com_x" value="0.058"  />
+	<xacro:property name="coxa_l"     value="0.06"  />
+	<xacro:property name="coxa_w"     value="0.06"  />
+	<xacro:property name="coxa_d"     value="0.055" />
+	<xacro:property name="coxa_cl"    value="0.03" />
+	<xacro:property name="coxa_com_x" value="0.02471"  />
 	<xacro:property name="coxa_com_y" value="0"  />
 	<xacro:property name="coxa_com_z" value="0"  />
-	<xacro:property name="coxa_m"     value="0.175" />
-	<xacro:property name="coxa_i_xx"  value="0.000032"  />
+	<xacro:property name="coxa_m"     value="0.0406" />
+	<xacro:property name="coxa_i_xx"  value="0.000038"  />
 	<xacro:property name="coxa_i_xy"  value="0.0"  />
 	<xacro:property name="coxa_i_xz"  value="0.0"  />
-	<xacro:property name="coxa_i_yy"  value="0.000056"  />
+	<xacro:property name="coxa_i_yy"  value="0.000038"  />
 	<xacro:property name="coxa_i_yz"  value="0.0"  />
-	<xacro:property name="coxa_i_zz"  value="0.00004"  />
+	<xacro:property name="coxa_i_zz"  value="0.000040"  />
 	<!-- Femur assembly -->
 	<xacro:property name="femur_l"     value="0.15" />
 	<xacro:property name="femur_w"     value="0.04" />
 	<xacro:property name="femur_d"     value="0.04" />
-	<xacro:property name="femur_cl"    value="0.12" />
-	<xacro:property name="femur_com_x" value="0.1213"  />
+	<xacro:property name="femur_cl"    value="0.15" />
+	<xacro:property name="femur_com_x" value="0.075"  />
 	<xacro:property name="femur_com_y" value="0"  />
 	<xacro:property name="femur_com_z" value="0"  />
-	<xacro:property name="femur_m"     value="0.1554" />
-	<xacro:property name="femur_i_xx"  value="0.000019"  />
+	<xacro:property name="femur_m"     value="0.35" />
+	<xacro:property name="femur_i_xx"  value="0.000014"  />
 	<xacro:property name="femur_i_xy"  value="0"  />
 	<xacro:property name="femur_i_xz"  value="0"  />
-	<xacro:property name="femur_i_yy"  value="0.000068"  />
+	<xacro:property name="femur_i_yy"  value="0.000047"  />
 	<xacro:property name="femur_i_yz"  value="0"  />
-	<xacro:property name="femur_i_zz"  value="0.000079"  />
+	<xacro:property name="femur_i_zz"  value="0.000051"  />
 	<!--  Tibia assembly -->
-	<xacro:property name="tibia_l" value="0.16" />
+	<xacro:property name="tibia_l" value="0.134" />
 	<xacro:property name="tibia_w" value="0.04" />
 	<xacro:property name="tibia_d" value="0.025" />
-	<xacro:property name="tibia_cl" value="0.12" />
-	<xacro:property name="tibia_com_x" value="0.0958"  	/>
+	<xacro:property name="tibia_cl" value="0.06" />
+	<xacro:property name="tibia_com_x" value="0.0887"  	/>
 	<xacro:property name="tibia_com_y" value="0"  		/>
 	<xacro:property name="tibia_com_z" value="0"  		/>
-	<xacro:property name="tibia_m"     value="0.0537" 	/>
-	<xacro:property name="tibia_i_xx"  value="0.000016" />
+	<xacro:property name="tibia_m"     value="0.076" 	/>
+	<xacro:property name="tibia_i_xx"  value="0.000025" />
 	<xacro:property name="tibia_i_xy"  value="0"  		/>
 	<xacro:property name="tibia_i_xz"  value="0"  		/>
-	<xacro:property name="tibia_i_yy"  value="0.000119" />
+	<xacro:property name="tibia_i_yy"  value="0.000105" />
 	<xacro:property name="tibia_i_yz"  value="0"  		/>
-	<xacro:property name="tibia_i_zz"  value="0.00013"  />
+	<xacro:property name="tibia_i_zz"  value="0.000117"  />
 	<!-- Foot -->
-	<xacro:property name="foot_r" value="0.008"   />
-	<xacro:property name="foot_m" value="0.005"   />
-	<xacro:property name="foot_I" value="0.00005" />
+	<xacro:property name="foot_r" value="0.016"   />
+	<xacro:property name="foot_m" value="0.040"   />
+	<xacro:property name="foot_I" value="0.000004" />
 	<!-- Rectangular box: m*(a^2 + b^2)/12 -->
 </robot>

File: mcorin_description/urdfs/leg/leg.xacro (robot description, xacro)
@@ -60,9 +60,9 @@
 		    </visual>
 		    <collision>
-		    	<origin rpy="0 0 0" xyz="0.05945 0 0"/>
-		      	<geometry>
-		        	<box size= "${coxa_cl} ${coxa_w} ${coxa_d}"/>
-		      	</geometry>
-		      	<material name="orange"/>
+		    	<origin rpy="0 0 0" xyz="0 0 0"/>
+			    <geometry>
+			      <mesh filename="package://mcorin_description/meshes/Coxa_collision.STL" scale="1 1 1"/>
+			    </geometry>
+		      <material name="orange"/>
 		    </collision>
 		    <inertial>
@@ -78,5 +78,5 @@
 		        	<mesh filename="package://mcorin_description/meshes/Femur.STL" scale="1 1 1"/>
 		      	</geometry>
-		      	<origin xyz="0 0 0" rpy="${pi/2} 0 0"/>
+		      	<origin xyz="0 0 0" rpy="0 0 0"/>
 		      	<material name="blue"/>
 		    </visual>
@@ -85,5 +85,5 @@
 		        	<box size= "${femur_cl} ${femur_w} ${femur_d}"/>
 		      	</geometry>
-		      	<origin xyz="0.1 0 0" rpy="0 0 0"/>
+		      	<origin xyz="0.075 0 0" rpy="0 0 0"/>
 		      	<material name="colli"/>
 		    </collision>
@@ -105,7 +105,8 @@
 		    <collision>
 		      	<geometry>
-		        	<box size= "${tibia_cl} ${tibia_d} ${tibia_w}"/>
+							<mesh filename="package://mcorin_description/meshes/Tibia_collision.STL" scale="1 1 1"/>
+		        	<!-- <box size= "${tibia_cl} ${tibia_d} ${tibia_w}"/> -->
 		      	</geometry>
-		      	<origin xyz="0.085 0 0" rpy="0 0 0"/>
+		      	<origin xyz="0.0 0 0" rpy="${pi/2} 0 0"/>
 		      	<material name="colli"/>
 		    </collision>

File: mcorin_description/urdfs/trunk/trunk_fixed.xacro (robot description, xacro)
@@ -25,5 +25,5 @@
 			<visual>
 				<geometry>
-					<box size= "${trunk_x} ${trunk_y} ${trunk_z}"/>
+					<mesh filename="package://mcorin_description/meshes/Body.STL" scale="1 1 1"/>
 				</geometry>
 				<material name="orange"/>
@@ -31,5 +31,5 @@
 			<collision>
 				<geometry>
-					<box size= "${trunk_x} ${trunk_y} ${trunk_z}"/>
+					<mesh filename="package://mcorin_description/meshes/Body_collision.STL" scale="1 1 1"/>
 				</geometry>
 				<material name="colli"/>
