Commit message: corIIn working with new dynamixel library, controllable via rosparam

File: mcorin_description/urdfs/trunk/trunk_model.xacro (robot description, xacro)
@@ -31,5 +31,6 @@
 			<visual>
 				<geometry>
-					<box size= "${trunk_x} ${trunk_y} ${trunk_z}"/>
+					<mesh filename="package://mcorin_description/meshes/Body.STL" scale="1 1 1"/>
+					<!-- <box size= "${trunk_x} ${trunk_y} ${trunk_z}"/> -->
 				</geometry>
 				<material name="orange"/>
@@ -37,5 +38,6 @@
 			<collision>
 				<geometry>
-					<box size= "${trunk_x} ${trunk_y} ${trunk_z}"/>
+					<mesh filename="package://mcorin_description/meshes/Body_collision.STL" scale="1 1 1"/>
+					<!-- <box size= "${trunk_x-0.02} ${3.8/5*trunk_y} ${trunk_z}"/> -->
 				</geometry>
 				<material name="colli"/>

Commit message: experimentation motion implemented,need finalisation with matlab data

File: mcorin_description/robots/fixed_mcorin.urdf (robot description, URDF)
Before this commit: robot corin, 27 links, 26 joints
Joints:
- joint base_qx_joint: origin xyz=0 0 -0.05 rpy=0 0 0 -> xyz=0 0 0.15 rpy=0 0 0
- joint lf_q1_joint: limit lower=-1.6 upper=1.6 effort=2.85 velocity=5.23 -> lower=-1.0 upper=1.0 effort=2.85 velocity=5.23
- joint lf_q2_joint: limit lower=-2.36 upper=2.36 effort=2.85 velocity=5.23 -> lower=-2.22 upper=2.22 effort=2.85 velocity=5.23
- joint lf_q3_joint: limit lower=-3.1 upper=3.1 effort=2.85 velocity=5.23 -> lower=-2.79 upper=2.79 effort=2.85 velocity=5.23
- joint lm_q1_joint: limit lower=-1.6 upper=1.6 effort=2.85 velocity=5.23 -> lower=-1.0 upper=1.0 effort=2.85 velocity=5.23
- joint lm_q2_joint: limit lower=-2.36 upper=2.36 effort=2.85 velocity=5.23 -> lower=-2.22 upper=2.22 effort=2.85 velocity=5.23
- joint lm_q3_joint: limit lower=-3.1 upper=3.1 effort=2.85 velocity=5.23 -> lower=-2.79 upper=2.79 effort=2.85 velocity=5.23
- joint lr_q1_joint: limit lower=-1.6 upper=1.6 effort=2.85 velocity=5.23 -> lower=-1.0 upper=1.0 effort=2.85 velocity=5.23
- joint lr_q2_joint: limit lower=-2.36 upper=2.36 effort=2.85 velocity=5.23 -> lower=-2.22 upper=2.22 effort=2.85 velocity=5.23
- joint lr_q3_joint: limit lower=-3.1 upper=3.1 effort=2.85 velocity=5.23 -> lower=-2.79 upper=2.79 effort=2.85 velocity=5.23
- joint rf_q1_joint: limit lower=-1.6 upper=1.6 effort=2.85 velocity=5.23 -> lower=-1.0 upper=1.0 effort=2.85 velocity=5.23
- joint rf_q2_joint: limit lower=-2.36 upper=2.36 effort=2.85 velocity=5.23 -> lower=-2.22 upper=2.22 effort=2.85 velocity=5.23
- joint rf_q3_joint: limit lower=-3.1 upper=3.1 effort=2.85 velocity=5.23 -> lower=-2.79 upper=2.79 effort=2.85 velocity=5.23
- joint rm_q1_joint: limit lower=-1.6 upper=1.6 effort=2.85 velocity=5.23 -> lower=-1.0 upper=1.0 effort=2.85 velocity=5.23
- joint rm_q2_joint: limit lower=-2.36 upper=2.36 effort=2.85 velocity=5.23 -> lower=-2.22 upper=2.22 effort=2.85 velocity=5.23
- joint rm_q3_joint: limit lower=-3.1 upper=3.1 effort=2.85 velocity=5.23 -> lower=-2.79 upper=2.79 effort=2.85 velocity=5.23
- joint rr_q1_joint: limit lower=-1.6 upper=1.6 effort=2.85 velocity=5.23 -> lower=-1.0 upper=1.0 effort=2.85 velocity=5.23
- joint rr_q2_joint: limit lower=-2.36 upper=2.36 effort=2.85 velocity=5.23 -> lower=-2.22 upper=2.22 effort=2.85 velocity=5.23
- joint rr_q3_joint: limit lower=-3.1 upper=3.1 effort=2.85 velocity=5.23 -> lower=-2.79 upper=2.79 effort=2.85 velocity=5.23

File: mcorin_description/urdfs/trunk/trunk_fixed.xacro (robot description, xacro)
@@ -9,5 +9,5 @@
 		<joint name="${name}_qx_joint" type="revolute">
 			<axis xyz="1 0 0"/>
-			<origin xyz="0 0 -0.05" rpy="0 0 0"/>
+			<origin xyz="0 0 0.15" rpy="0 0 0"/>
 			<limit effort="30." velocity="2.0" lower="-0.001" upper="0.001"/>
 			<dynamics damping="0.3" friction="0" />
