Commit message: resolved leg flipping backwards, working on node to control leg manually

File: mcorin_description/robots/mCorin_model.urdf.xacro (robot description, xacro)
@@ -28,4 +28,5 @@
 		name="lf"
 		parent="trunk"
+		middle_leg="false"
 		load_force_sensors="true">
 		<origin xyz="${trunk_x/2} ${trunk_y/2} 0" rpy="0 0 ${50*PI/180}"/>
@@ -34,4 +35,5 @@
 		name="lm"
 		parent="trunk"
+		middle_leg="true"
 		load_force_sensors="false">
 		<origin xyz="0 ${trunk_y/2} 0" rpy="0 0 ${PI/2}"/>
@@ -40,4 +42,5 @@
 		name="lr"
 		parent="trunk"
+		middle_leg="false"
 		load_force_sensors="false">
 		<origin xyz="${-trunk_x/2} ${trunk_y/2} 0" rpy="0 0 ${PI/2+40*PI/180}"/>
@@ -46,4 +49,5 @@
 		name="rf"
 		parent="trunk"
+		middle_leg="false"
 		load_force_sensors="true">
 		<origin xyz="${trunk_x/2} ${-trunk_y/2} 0" rpy="0 0 ${-50*PI/180}"/>
@@ -52,4 +56,5 @@
 		name="rm"
 		parent="trunk"
+		middle_leg="true"
 		load_force_sensors="false">
 		<origin xyz="0 ${-trunk_y/2} 0" rpy="0 0 ${-PI/2}"/>
@@ -58,4 +63,5 @@
 		name="rr"
 		parent="trunk"
+		middle_leg="false"
 		load_force_sensors="false">
 		<origin xyz="${-trunk_x/2} ${-trunk_y/2} 0" rpy="0 0 ${-PI/2-40*PI/180}"/>

File: mcorin_description/robots/mcorin.urdf (robot description, URDF)
Before this commit: robot corin, 28 links, 27 joints
Links:
- link lf_foot: mass 0.005 -> 0.04
- link lf_hipassembly: mass 0.175 -> 0.0406
- link lf_lowerleg: mass 0.0537 -> 0.076
- link lf_upperleg: mass 0.1554 -> 0.35
- link lm_foot: mass 0.005 -> 0.04
- link lm_hipassembly: mass 0.175 -> 0.0406
- link lm_lowerleg: mass 0.0537 -> 0.076
- link lm_upperleg: mass 0.1554 -> 0.35
- link lr_foot: mass 0.005 -> 0.04
- link lr_hipassembly: mass 0.175 -> 0.0406
- link lr_lowerleg: mass 0.0537 -> 0.076
- link lr_upperleg: mass 0.1554 -> 0.35
- link rf_foot: mass 0.005 -> 0.04
- link rf_hipassembly: mass 0.175 -> 0.0406
- link rf_lowerleg: mass 0.0537 -> 0.076
- link rf_upperleg: mass 0.1554 -> 0.35
- link rm_foot: mass 0.005 -> 0.04
- link rm_hipassembly: mass 0.175 -> 0.0406
- link rm_lowerleg: mass 0.0537 -> 0.076
- link rm_upperleg: mass 0.1554 -> 0.35
- link rr_foot: mass 0.005 -> 0.04
- link rr_hipassembly: mass 0.175 -> 0.0406
- link rr_lowerleg: mass 0.0537 -> 0.076
- link rr_upperleg: mass 0.1554 -> 0.35
- link trunk: mass 1.5 -> 1.58
Joints:
- joint lf_q1_joint: limit lower=-1.6 upper=1.6 effort=2.85 velocity=5.23 -> lower=-1.0 upper=1.0 effort=2.85 velocity=5.23
- joint lf_q2_joint: limit lower=-2.36 upper=2.36 effort=2.85 velocity=5.23 -> lower=-2.22 upper=2.22 effort=2.85 velocity=5.23
- joint lf_q3_joint: limit lower=-3.1 upper=3.1 effort=2.85 velocity=5.23 -> lower=-2.79 upper=2.79 effort=2.85 velocity=5.23
- joint lm_q1_joint: limit lower=-1.6 upper=1.6 effort=2.85 velocity=5.23 -> lower=-0.84 upper=0.84 effort=2.85 velocity=5.23
- joint lm_q2_joint: limit lower=-2.36 upper=2.36 effort=2.85 velocity=5.23 -> lower=-2.22 upper=2.22 effort=2.85 velocity=5.23
- joint lm_q3_joint: limit lower=-3.1 upper=3.1 effort=2.85 velocity=5.23 -> lower=-2.79 upper=2.79 effort=2.85 velocity=5.23
- joint lr_q1_joint: limit lower=-1.6 upper=1.6 effort=2.85 velocity=5.23 -> lower=-1.0 upper=1.0 effort=2.85 velocity=5.23
- joint lr_q2_joint: limit lower=-2.36 upper=2.36 effort=2.85 velocity=5.23 -> lower=-2.22 upper=2.22 effort=2.85 velocity=5.23
- joint lr_q3_joint: limit lower=-3.1 upper=3.1 effort=2.85 velocity=5.23 -> lower=-2.79 upper=2.79 effort=2.85 velocity=5.23
- joint rf_q1_joint: limit lower=-1.6 upper=1.6 effort=2.85 velocity=5.23 -> lower=-1.0 upper=1.0 effort=2.85 velocity=5.23
- joint rf_q2_joint: limit lower=-2.36 upper=2.36 effort=2.85 velocity=5.23 -> lower=-2.22 upper=2.22 effort=2.85 velocity=5.23
- joint rf_q3_joint: limit lower=-3.1 upper=3.1 effort=2.85 velocity=5.23 -> lower=-2.79 upper=2.79 effort=2.85 velocity=5.23
- joint rm_q1_joint: limit lower=-1.6 upper=1.6 effort=2.85 velocity=5.23 -> lower=-0.84 upper=0.84 effort=2.85 velocity=5.23
- joint rm_q2_joint: limit lower=-2.36 upper=2.36 effort=2.85 velocity=5.23 -> lower=-2.22 upper=2.22 effort=2.85 velocity=5.23
- joint rm_q3_joint: limit lower=-3.1 upper=3.1 effort=2.85 velocity=5.23 -> lower=-2.79 upper=2.79 effort=2.85 velocity=5.23
- joint rr_q1_joint: limit lower=-1.6 upper=1.6 effort=2.85 velocity=5.23 -> lower=-1.0 upper=1.0 effort=2.85 velocity=5.23
- joint rr_q2_joint: limit lower=-2.36 upper=2.36 effort=2.85 velocity=5.23 -> lower=-2.22 upper=2.22 effort=2.85 velocity=5.23
- joint rr_q3_joint: limit lower=-3.1 upper=3.1 effort=2.85 velocity=5.23 -> lower=-2.79 upper=2.79 effort=2.85 velocity=5.23

File: mcorin_description/urdfs/leg/leg.xacro (robot description, xacro)
@@ -6,5 +6,5 @@
 	<!-- ================================== Leg ================================== -->
 	<!-- The xacro macro xacro:mcorin_leg contains: hip assembly, upper and lower leg -->
-	<xacro:macro name="mCorin_leg" params="name parent *origin load_force_sensors">
+	<xacro:macro name="mCorin_leg" params="name parent middle_leg *origin load_force_sensors">
 		<!-- Joints -->
 		<!-- Coxa joint -->
@@ -14,5 +14,10 @@
 			<child  link="${name}_hipassembly"/>
 			<axis xyz="0 0 1"/>
-			<limit effort="${MX64_effort}" velocity="${MX64_velocity}" lower="${-cox_joint_lim}" upper="${cox_joint_lim}"/>
+			<xacro:if value="${middle_leg}"> 	<!-- overwrite joint limits for middle legs-->
+				<limit effort="${MX64_effort}" velocity="${MX64_velocity}" lower="${-cxm_joint_lim}" upper="${cxm_joint_lim}"/>
+			</xacro:if>
+			<xacro:unless value="${middle_leg}"> 	<!-- overwrite joint limits for middle legs-->
+				<limit effort="${MX64_effort}" velocity="${MX64_velocity}" lower="${-cox_joint_lim}" upper="${cox_joint_lim}"/>
+			</xacro:unless>
 			<dynamics damping="${MX64_damping}" friction="0" />
 			<!-- <safety_controller k_position="100" k_velocity="100"
