Commit message: currently working on local HP desktop, prior to spline modification

File: mcorin_description/robots/mcorin.urdf (robot description, URDF)
Before this commit: robot corin, 29 links, 28 joints
Joints:
- joint lf_q1_joint: limit lower=-1.0 upper=1.0 effort=5.0 velocity=5.23 -> lower=-1.0 upper=1.0 effort=2.85 velocity=5.23
- joint lf_q2_joint: limit lower=-2.22 upper=2.22 effort=5.0 velocity=5.23 -> lower=-2.22 upper=2.22 effort=2.85 velocity=5.23
- joint lf_q3_joint: limit lower=-2.79 upper=2.79 effort=5.0 velocity=5.23 -> lower=-2.79 upper=2.79 effort=2.85 velocity=5.23
- joint lm_q1_joint: limit lower=-0.84 upper=0.84 effort=5.0 velocity=5.23 -> lower=-0.84 upper=0.84 effort=2.85 velocity=5.23
- joint lm_q2_joint: limit lower=-2.22 upper=2.22 effort=5.0 velocity=5.23 -> lower=-2.22 upper=2.22 effort=2.85 velocity=5.23
- joint lm_q3_joint: limit lower=-2.79 upper=2.79 effort=5.0 velocity=5.23 -> lower=-2.79 upper=2.79 effort=2.85 velocity=5.23
- joint lr_q1_joint: limit lower=-1.0 upper=1.0 effort=5.0 velocity=5.23 -> lower=-1.0 upper=1.0 effort=2.85 velocity=5.23
- joint lr_q2_joint: limit lower=-2.22 upper=2.22 effort=5.0 velocity=5.23 -> lower=-2.22 upper=2.22 effort=2.85 velocity=5.23
- joint lr_q3_joint: limit lower=-2.79 upper=2.79 effort=5.0 velocity=5.23 -> lower=-2.79 upper=2.79 effort=2.85 velocity=5.23
- joint rf_q1_joint: limit lower=-1.0 upper=1.0 effort=5.0 velocity=5.23 -> lower=-1.0 upper=1.0 effort=2.85 velocity=5.23
- joint rf_q2_joint: limit lower=-2.22 upper=2.22 effort=5.0 velocity=5.23 -> lower=-2.22 upper=2.22 effort=2.85 velocity=5.23
- joint rf_q3_joint: limit lower=-2.79 upper=2.79 effort=5.0 velocity=5.23 -> lower=-2.79 upper=2.79 effort=2.85 velocity=5.23
- joint rm_q1_joint: limit lower=-0.84 upper=0.84 effort=5.0 velocity=5.23 -> lower=-0.84 upper=0.84 effort=2.85 velocity=5.23
- joint rm_q2_joint: limit lower=-2.22 upper=2.22 effort=5.0 velocity=5.23 -> lower=-2.22 upper=2.22 effort=2.85 velocity=5.23
- joint rm_q3_joint: limit lower=-2.79 upper=2.79 effort=5.0 velocity=5.23 -> lower=-2.79 upper=2.79 effort=2.85 velocity=5.23
- joint rr_q1_joint: limit lower=-1.0 upper=1.0 effort=5.0 velocity=5.23 -> lower=-1.0 upper=1.0 effort=2.85 velocity=5.23
- joint rr_q2_joint: limit lower=-2.22 upper=2.22 effort=5.0 velocity=5.23 -> lower=-2.22 upper=2.22 effort=2.85 velocity=5.23
- joint rr_q3_joint: limit lower=-2.79 upper=2.79 effort=5.0 velocity=5.23 -> lower=-2.79 upper=2.79 effort=2.85 velocity=5.23

File: mcorin_description/urdfs/common.xacro (robot description, xacro)
@@ -8,5 +8,5 @@
 	<!--  Joint parameters -->
 	<xacro:property name="MX64_damping"   value="0.15" /> 					<!-- real: 0.2 		-->
-	<xacro:property name="MX64_effort"    value="5.0" /> 					<!-- real: 2.85 Nm 	-->
+	<xacro:property name="MX64_effort"    value="2.85" /> 					<!-- real: 2.85 Nm 	-->
 	<xacro:property name="MX64_velocity"  value="5.23" />
 	<xacro:property name="cox_joint_lim" value="1.00" />	<!-- 57deg -->
