Commit message: hardware now visualised on rviz;hardware joint name changed to include _joint

File: mcorin_description/robots/mCorin_fixed.urdf.xacro (robot description, xacro)
@@ -65,8 +65,16 @@
 		parent="trunk"
 		imu_name="trunk_imu"
-		imu_topic="trunk/data"
+		imu_topic="middle/data"
 		imu_service="trunk/service"
 		update_rate="100">
 		<origin xyz="0.0 0.0 0.0" rpy="0 0 0"/>
+	</xacro:IMU>
+	<xacro:IMU
+		parent="trunk"
+		imu_name="trunk_offset_imu"
+		imu_topic="offset/data"
+		imu_service="trunk/service2"
+		update_rate="100">
+		<origin xyz="0.0 0.0 0.022" rpy="0 0 0"/>
 	</xacro:IMU>
 	<!-- <xacro:LIDAR

File: mcorin_description/robots/mCorin_model.urdf.xacro (robot description, xacro)
@@ -71,8 +71,16 @@
 		parent="trunk"
 		imu_name="trunk_imu"
-		imu_topic="trunk/data"
+		imu_topic="middle/data"
 		imu_service="trunk/service"
 		update_rate="100">
 		<origin xyz="0.0 0.0 0.0" rpy="0 0 0"/>
+	</xacro:IMU>
+	<xacro:IMU
+		parent="trunk"
+		imu_name="trunk_offset_imu"
+		imu_topic="offset/data"
+		imu_service="trunk/service2"
+		update_rate="100">
+		<origin xyz="0.0 0.0 0.022" rpy="0 0 0"/>
 	</xacro:IMU>
 	<xacro:LIDAR

File: mcorin_description/robots/mcorin.urdf (robot description, URDF)
Before this commit: robot corin, 28 links, 27 joints
Links:
- added link trunk_offset_imu, mass 0.010; visual box size=0.05 0.05 0.01
Joints:
- added joint trunk_offset_imu_joint: type fixed, parent trunk, child trunk_offset_imu, origin xyz=0.0 0.0 0.022 rpy=0 0 0
- joint lf_q1_joint: limit lower=-1.0 upper=1.0 effort=2.85 velocity=5.23 -> lower=-1.0 upper=1.0 effort=5.0 velocity=5.23
- joint lf_q2_joint: limit lower=-2.22 upper=2.22 effort=2.85 velocity=5.23 -> lower=-2.22 upper=2.22 effort=5.0 velocity=5.23
- joint lf_q3_joint: limit lower=-2.79 upper=2.79 effort=2.85 velocity=5.23 -> lower=-2.79 upper=2.79 effort=5.0 velocity=5.23
- joint lm_q1_joint: limit lower=-0.84 upper=0.84 effort=2.85 velocity=5.23 -> lower=-0.84 upper=0.84 effort=5.0 velocity=5.23
- joint lm_q2_joint: limit lower=-2.22 upper=2.22 effort=2.85 velocity=5.23 -> lower=-2.22 upper=2.22 effort=5.0 velocity=5.23
- joint lm_q3_joint: limit lower=-2.79 upper=2.79 effort=2.85 velocity=5.23 -> lower=-2.79 upper=2.79 effort=5.0 velocity=5.23
- joint lr_q1_joint: limit lower=-1.0 upper=1.0 effort=2.85 velocity=5.23 -> lower=-1.0 upper=1.0 effort=5.0 velocity=5.23
- joint lr_q2_joint: limit lower=-2.22 upper=2.22 effort=2.85 velocity=5.23 -> lower=-2.22 upper=2.22 effort=5.0 velocity=5.23
- joint lr_q3_joint: limit lower=-2.79 upper=2.79 effort=2.85 velocity=5.23 -> lower=-2.79 upper=2.79 effort=5.0 velocity=5.23
- joint rf_q1_joint: limit lower=-1.0 upper=1.0 effort=2.85 velocity=5.23 -> lower=-1.0 upper=1.0 effort=5.0 velocity=5.23
- joint rf_q2_joint: limit lower=-2.22 upper=2.22 effort=2.85 velocity=5.23 -> lower=-2.22 upper=2.22 effort=5.0 velocity=5.23
- joint rf_q3_joint: limit lower=-2.79 upper=2.79 effort=2.85 velocity=5.23 -> lower=-2.79 upper=2.79 effort=5.0 velocity=5.23
- joint rm_q1_joint: limit lower=-0.84 upper=0.84 effort=2.85 velocity=5.23 -> lower=-0.84 upper=0.84 effort=5.0 velocity=5.23
- joint rm_q2_joint: limit lower=-2.22 upper=2.22 effort=2.85 velocity=5.23 -> lower=-2.22 upper=2.22 effort=5.0 velocity=5.23
- joint rm_q3_joint: limit lower=-2.79 upper=2.79 effort=2.85 velocity=5.23 -> lower=-2.79 upper=2.79 effort=5.0 velocity=5.23
- joint rr_q1_joint: limit lower=-1.0 upper=1.0 effort=2.85 velocity=5.23 -> lower=-1.0 upper=1.0 effort=5.0 velocity=5.23
- joint rr_q2_joint: limit lower=-2.22 upper=2.22 effort=2.85 velocity=5.23 -> lower=-2.22 upper=2.22 effort=5.0 velocity=5.23
- joint rr_q3_joint: limit lower=-2.79 upper=2.79 effort=2.85 velocity=5.23 -> lower=-2.79 upper=2.79 effort=5.0 velocity=5.23

File: mcorin_description/urdfs/common.xacro (robot description, xacro)
@@ -8,5 +8,5 @@
 	<!--  Joint parameters -->
 	<xacro:property name="MX64_damping"   value="0.15" /> 					<!-- real: 0.2 		-->
-	<xacro:property name="MX64_effort"    value="2.85" /> 					<!-- real: 2.85 Nm 	-->
+	<xacro:property name="MX64_effort"    value="5.0" /> 					<!-- real: 2.85 Nm 	-->
 	<xacro:property name="MX64_velocity"  value="5.23" />
 	<xacro:property name="cox_joint_lim" value="1.00" />	<!-- 57deg -->

Commit message: offload dxl rad2raw to RobotisFramework; tidied up robot_controller(previously controller_walking);

File: mcorin_description/robots/mCorin_fixed.urdf.xacro (robot description, xacro)
@@ -28,4 +28,5 @@
 		name="lf"
 		parent="trunk"
+		middle_leg="false"
 		load_force_sensors="true">
 		<origin xyz="${trunk_x/2} ${trunk_y/2} 0" rpy="0 0 ${50*PI/180}"/>
@@ -34,4 +35,5 @@
 		name="lm"
 		parent="trunk"
+		middle_leg="true"
 		load_force_sensors="false">
 		<origin xyz="0 ${trunk_y/2} 0" rpy="0 0 ${PI/2}"/>
@@ -40,4 +42,5 @@
 		name="lr"
 		parent="trunk"
+		middle_leg="false"
 		load_force_sensors="false">
 		<origin xyz="${-trunk_x/2} ${trunk_y/2} 0" rpy="0 0 ${PI/2+40*PI/180}"/>
@@ -46,4 +49,5 @@
 		name="rf"
 		parent="trunk"
+		middle_leg="false"
 		load_force_sensors="true">
 		<origin xyz="${trunk_x/2} ${-trunk_y/2} 0" rpy="0 0 ${-50*PI/180}"/>
@@ -52,4 +56,5 @@
 		name="rm"
 		parent="trunk"
+		middle_leg="true"
 		load_force_sensors="false">
 		<origin xyz="0 ${-trunk_y/2} 0" rpy="0 0 ${-PI/2}"/>
@@ -58,4 +63,5 @@
 		name="rr"
 		parent="trunk"
+		middle_leg="false"
 		load_force_sensors="false">
 		<origin xyz="${-trunk_x/2} ${-trunk_y/2} 0" rpy="0 0 ${-PI/2-40*PI/180}"/>
@@ -78,10 +84,10 @@
 		<origin xyz="0.0 0.0 0.022" rpy="0 0 0"/>
 	</xacro:IMU>
-	<!-- <xacro:LIDAR
+	<xacro:LIDAR
 		parent="trunk"
 		lidar_name="trunk_lidar"
 		lidar_topic="lidar/data"
 		update_rate="100">
-		<origin xyz="0.12 0.0 0.03" rpy="0 0 0"/>
-	</xacro:LIDAR> -->
+		<origin xyz="0.06 0.0 0.04" rpy="0 0 ${PI/2}"/>
+	</xacro:LIDAR>
 </robot>
