Commit message: Integrated state estimator

File: corin_description/robots/Corin_model.urdf.xacro (robot description, xacro)
@@ -65,6 +65,6 @@
 		imu_topic="base/data"
 		imu_service="trunk/service"
-		update_rate="100">
-		<origin xyz="0.0 0.0 0.022" rpy="0 0 0"/>
+		freq_rate="200">
+		<origin xyz="0.0 0.0 0.0" rpy="0 0 0"/><!-- 0.022-->
 	</xacro:IMU>
 	<!--

File: corin_description/urdfs/sensors/sensors.xacro (robot description, xacro)
@@ -2,5 +2,5 @@
 <robot xmlns:xacro="http://www.ros.org/wiki/xacro" name="corin">
 	<!-- #############  IMU Sensor  ############# -->
-	<xacro:macro name="IMU" params="parent imu_name imu_topic imu_service update_rate *origin">
+	<xacro:macro name="IMU" params="parent imu_name imu_topic imu_service freq_rate *origin">
         <!-- Joint -->
         <joint name="${imu_name}_joint" type="fixed">
@@ -26,16 +26,26 @@
             </visual>
         </link>
-        <gazebo>
-            <material>Gazebo/Red</material>
-            <plugin name="imu_plugin" filename="libgazebo_ros_imu.so">
-                <robotNamespace>/corin/imu/</robotNamespace>
-                <alwaysOn>true</alwaysOn>
-                <frameName>${imu_name}</frameName>
-                <bodyName>${imu_name}</bodyName>
+				<gazebo reference="${imu_name}">
+					<material>Gazebo/Red</material>
+					<gravity>false</gravity>
+					<sensor name='IMU' type='imu'>
+						<always_on>true</always_on>
+						<!-- <update_rate>${freq_rate}</update_rate> -->
+						<visualize>true</visualize>
+						<topic>__default_topic__</topic>
+            <plugin name="imu_plugin" filename="libgazebo_ros_imu_sensor.so">
+								<robotNamespace>/corin/imu/</robotNamespace>
+								<alwaysOn>true</alwaysOn>
+								<gravity>false</gravity>
+								<frameName>${imu_name}</frameName>
                 <topicName>${imu_topic}</topicName>
                 <serviceName>${imu_service}</serviceName>
-                <gaussianNoise>0.1</gaussianNoise>
-                <updateRate>${update_rate}</updateRate>
+								<bodyName>${imu_name}</bodyName>
+                <updateRateHZ>${freq_rate}</updateRateHZ>
+								<gaussianNoise>0</gaussianNoise>
+								<xyzOffset>0 0 0</xyzOffset>
+    						<rpyOffset>0 0 0</rpyOffset>
             </plugin>
+					</sensor>
         </gazebo>
     </xacro:macro>

Commit message: Modified sensor model

File: corin_description/robots/Corin_model.urdf.xacro (robot description, xacro)
@@ -60,5 +60,5 @@
 	</xacro:RobotLeg>
 	<!-- Sensors -->
-	<xacro:IMU
+	<!-- <xacro:IMU
 		parent="trunk"
 		imu_name="base_imu"
@@ -67,4 +67,12 @@
 		update_rate="100">
 		<origin xyz="0.0 0.0 0.022" rpy="0 0 0"/>
+	</xacro:IMU> -->
+	<xacro:IMU
+		parent="trunk"
+		imu_name="base_imu"
+		imu_topic="base/data"
+		imu_service="trunk/service"
+		freq_rate="200">
+		<origin xyz="0 0 0.0" rpy="0 0 0"/>
 	</xacro:IMU>
 	<!--

File: corin_description/urdfs/sensors/sensors_old.xacro (robot description, xacro)
@@ -2,5 +2,5 @@
 <robot xmlns:xacro="http://www.ros.org/wiki/xacro" name="corin">
 	<!-- #############  IMU Sensor  ############# -->
-	<xacro:macro name="IMU" params="parent imu_name imu_topic imu_service freq_rate *origin">
+	<xacro:macro name="IMU" params="parent imu_name imu_topic imu_service update_rate *origin">
         <!-- Joint -->
         <joint name="${imu_name}_joint" type="fixed">
@@ -12,6 +12,6 @@
         <link name="${imu_name}">
             <inertial>
-                <origin xyz="-0.0000  0.0000  0.000"/>
-                <mass value="0.0000"/>
+                <origin xyz="-0.00020  0.00010  0.00110"/>
+                <mass value="0.010"/>
                 <inertia ixx="0.0" iyy="0.0" izz="0.0" ixy="0.0" ixz="0.0" iyz="0.0"/>
             </inertial>
@@ -19,5 +19,5 @@
                 <origin xyz="0.0 0 0.0" rpy="0 0 0"/>
                 <geometry>
-                    <box size="0.05 0.1 0.01" />
+                    <box size="0.05 0.05 0.01" />
                 </geometry>
                 <material name="black">
@@ -25,37 +25,17 @@
                 </material>
             </visual>
-						<collision>
-								<origin xyz="0.0 0 0.0" rpy="0 0 0"/>
-								<geometry>
-										<box size="0.05 0.1 0.01" />
-								</geometry>
-								<material name="black">
-										<color rgba="0 0 0 0.9"/>
-								</material>
-						</collision>
         </link>
-        <gazebo reference="${imu_name}">
-					<material>Gazebo/Red</material>
-					<gravity>false</gravity>
-					<sensor name='IMU' type='imu'>
-						<always_on>true</always_on>
-						<!-- <update_rate>${freq_rate}</update_rate> -->
-						<visualize>true</visualize>
-						<topic>__default_topic__</topic>
-            <plugin name="imu_plugin" filename="libgazebo_ros_imu_sensor.so">
-								<robotNamespace>/corin/imu/</robotNamespace>
-								<alwaysOn>true</alwaysOn>
-								<gravity>false</gravity>
-								<frameName>${imu_name}</frameName>
+        <gazebo>
+            <material>Gazebo/Red</material>
+            <plugin name="imu_plugin" filename="libgazebo_ros_imu.so">
+                <robotNamespace>/corin/imu/</robotNamespace>
+                <alwaysOn>true</alwaysOn>
+                <frameName>${imu_name}</frameName>
+                <bodyName>${imu_name}</bodyName>
                 <topicName>${imu_topic}</topicName>
                 <serviceName>${imu_service}</serviceName>
-								<bodyName>${imu_name}</bodyName>
-                <updateRateHZ>${freq_rate}</updateRateHZ>
-								<gaussianNoise>0</gaussianNoise>
-								<xyzOffset>0 0 0</xyzOffset>
-    						<rpyOffset>0 0 0</rpyOffset>
+                <gaussianNoise>0.1</gaussianNoise>
+                <updateRate>${update_rate}</updateRate>
             </plugin>
-						<pose>0 0 0 0 0 0</pose>
-					</sensor>
         </gazebo>
     </xacro:macro>
