Commit message: using new transform library, path tracking inaccurate

File: corin_description/robots/Corin_fixed.urdf.xacro (robot description, xacro)
@@ -22,8 +22,8 @@
 	<!-- body -->
 	<!-- trunk -->
-	<xacro:mCorin_trunk name="base">
+	<xacro:RobotTrunk name="base">
 		<origin xyz="0.0 0.0 0.0" rpy="0 0 0"/>
-	</xacro:mCorin_trunk>
-	<xacro:mCorin_leg
+	</xacro:RobotTrunk>
+	<xacro:RobotLeg
 		name="lf"
 		parent="trunk"
@@ -31,6 +31,6 @@
 		load_force_sensors="true">
 		<origin xyz="${trunk_x/2} ${trunk_y/2} 0" rpy="0 0 ${50*PI/180}"/>
-	</xacro:mCorin_leg>
-	<xacro:mCorin_leg
+	</xacro:RobotLeg>
+	<xacro:RobotLeg
 		name="lm"
 		parent="trunk"
@@ -38,6 +38,6 @@
 		load_force_sensors="false">
 		<origin xyz="0 ${trunk_y/2} 0" rpy="0 0 ${PI/2}"/>
-	</xacro:mCorin_leg>
-	<xacro:mCorin_leg
+	</xacro:RobotLeg>
+	<xacro:RobotLeg
 		name="lr"
 		parent="trunk"
@@ -45,6 +45,6 @@
 		load_force_sensors="false">
 		<origin xyz="${-trunk_x/2} ${trunk_y/2} 0" rpy="0 0 ${PI/2+40*PI/180}"/>
-	</xacro:mCorin_leg>
-	<xacro:mCorin_leg
+	</xacro:RobotLeg>
+	<xacro:RobotLeg
 		name="rf"
 		parent="trunk"
@@ -52,6 +52,6 @@
 		load_force_sensors="true">
 		<origin xyz="${trunk_x/2} ${-trunk_y/2} 0" rpy="0 0 ${-50*PI/180}"/>
-	</xacro:mCorin_leg>
-	<xacro:mCorin_leg
+	</xacro:RobotLeg>
+	<xacro:RobotLeg
 		name="rm"
 		parent="trunk"
@@ -59,6 +59,6 @@
 		load_force_sensors="false">
 		<origin xyz="0 ${-trunk_y/2} 0" rpy="0 0 ${-PI/2}"/>
-	</xacro:mCorin_leg>
-	<xacro:mCorin_leg
+	</xacro:RobotLeg>
+	<xacro:RobotLeg
 		name="rr"
 		parent="trunk"
@@ -66,19 +66,11 @@
 		load_force_sensors="false">
 		<origin xyz="${-trunk_x/2} ${-trunk_y/2} 0" rpy="0 0 ${-PI/2-40*PI/180}"/>
-	</xacro:mCorin_leg>
+	</xacro:RobotLeg>
 	<!-- Sensors -->
 	<xacro:IMU
 		parent="trunk"
-		imu_name="trunk_imu"
-		imu_topic="middle/data"
+		imu_name="base_imu"
+		imu_topic="base/data"
 		imu_service="trunk/service"
-		update_rate="100">
-		<origin xyz="0.0 0.0 0.0" rpy="0 0 0"/>
-	</xacro:IMU>
-	<xacro:IMU
-		parent="trunk"
-		imu_name="trunk_offset_imu"
-		imu_topic="offset/data"
-		imu_service="trunk/service2"
 		update_rate="100">
 		<origin xyz="0.0 0.0 0.022" rpy="0 0 0"/>

File: corin_description/robots/Corin_model.urdf.xacro (robot description, xacro)
@@ -21,9 +21,8 @@
 is the world frame). For more, see http://www.ros.org/wiki/xacro -->
 	<!-- body -->
-	<!-- trunk -->
-	<xacro:mCorin_trunk name="base">
+	<xacro:RobotTrunk name="base">
 		<origin xyz="0.0 0.0 0.0" rpy="0 0 0"/>
-	</xacro:mCorin_trunk>
-	<xacro:mCorin_leg
+	</xacro:RobotTrunk>
+	<xacro:RobotLeg
 		name="lf"
 		parent="trunk"
@@ -31,6 +30,6 @@
 		load_force_sensors="true">
 		<origin xyz="${trunk_x/2} ${trunk_y/2} 0" rpy="0 0 ${50*PI/180}"/>
-	</xacro:mCorin_leg>
-	<xacro:mCorin_leg
+	</xacro:RobotLeg>
+	<xacro:RobotLeg
 		name="lm"
 		parent="trunk"
@@ -38,6 +37,6 @@
 		load_force_sensors="false">
 		<origin xyz="0 ${trunk_y/2} 0" rpy="0 0 ${PI/2}"/>
-	</xacro:mCorin_leg>
-	<xacro:mCorin_leg
+	</xacro:RobotLeg>
+	<xacro:RobotLeg
 		name="lr"
 		parent="trunk"
@@ -45,6 +44,6 @@
 		load_force_sensors="false">
 		<origin xyz="${-trunk_x/2} ${trunk_y/2} 0" rpy="0 0 ${PI/2+40*PI/180}"/>
-	</xacro:mCorin_leg>
-	<xacro:mCorin_leg
+	</xacro:RobotLeg>
+	<xacro:RobotLeg
 		name="rf"
 		parent="trunk"
@@ -52,6 +51,6 @@
 		load_force_sensors="true">
 		<origin xyz="${trunk_x/2} ${-trunk_y/2} 0" rpy="0 0 ${-50*PI/180}"/>
-	</xacro:mCorin_leg>
-	<xacro:mCorin_leg
+	</xacro:RobotLeg>
+	<xacro:RobotLeg
 		name="rm"
 		parent="trunk"
@@ -59,6 +58,6 @@
 		load_force_sensors="false">
 		<origin xyz="0 ${-trunk_y/2} 0" rpy="0 0 ${-PI/2}"/>
-	</xacro:mCorin_leg>
-	<xacro:mCorin_leg
+	</xacro:RobotLeg>
+	<xacro:RobotLeg
 		name="rr"
 		parent="trunk"
@@ -66,19 +65,11 @@
 		load_force_sensors="false">
 		<origin xyz="${-trunk_x/2} ${-trunk_y/2} 0" rpy="0 0 ${-PI/2-40*PI/180}"/>
-	</xacro:mCorin_leg>
+	</xacro:RobotLeg>
 	<!-- Sensors -->
 	<xacro:IMU
 		parent="trunk"
-		imu_name="trunk_imu"
-		imu_topic="middle/data"
+		imu_name="base_imu"
+		imu_topic="base/data"
 		imu_service="trunk/service"
-		update_rate="100">
-		<origin xyz="0.0 0.0 0.0" rpy="0 0 0"/>
-	</xacro:IMU>
-	<xacro:IMU
-		parent="trunk"
-		imu_name="trunk_offset_imu"
-		imu_topic="offset/data"
-		imu_service="trunk/service2"
 		update_rate="100">
 		<origin xyz="0.0 0.0 0.022" rpy="0 0 0"/>

File: corin_description/urdfs/leg/leg.xacro (robot description, xacro)
@@ -6,5 +6,5 @@
 	<!-- ================================== Leg ================================== -->
 	<!-- The xacro macro xacro:corin_leg contains: hip assembly, upper and lower leg -->
-	<xacro:macro name="mCorin_leg" params="name parent middle_leg *origin load_force_sensors">
+	<xacro:macro name="RobotLeg" params="name parent middle_leg *origin load_force_sensors">
 		<!-- Joints -->
 		<!-- Coxa joint -->

File: corin_description/urdfs/trunk/trunk_fixed.xacro (robot description, xacro)
@@ -5,5 +5,5 @@
 	<link name="world"/>
 	<!-- ================================ Trunk ================================ -->
-	<xacro:macro name="mCorin_trunk" params="name *origin">
+	<xacro:macro name="RobotTrunk" params="name *origin">
 		<!-- Floating-base Joint -->
 		<joint name="${name}_qx_joint" type="revolute">

File: corin_description/urdfs/trunk/trunk_model.xacro (robot description, xacro)
@@ -4,5 +4,5 @@
 	<xacro:include filename="$(find corin_description)/urdfs/trunk/trunk.gazebo.xacro"/>
 	<!-- ================================ Trunk ================================ -->
-	<xacro:macro name="mCorin_trunk" params="name *origin">
+	<xacro:macro name="RobotTrunk" params="name *origin">
 		<!-- Floating-base Joint -->
 		<joint name="floating_base" type="fixed">

Commit message: tuning admittance controller

File: corin_description/robots/Corin_fixed.urdf.xacro (robot description, xacro)
@@ -15,5 +15,5 @@
 	<!-- body -->
 	<xacro:RobotTrunk name="base">
-		<origin xyz="0.0 0.0 0.0" rpy="0 0 0"/>
+		<origin xyz="0 0 0" rpy="0 0 0"/>
 	</xacro:RobotTrunk>
 	<xacro:RobotLeg
