Commit message: impedance tuning in progress;gait phase update incorrect

File: corin_description/urdfs/trunk/trunk_fixed.xacro (robot description, xacro)
@@ -7,9 +7,9 @@
 	<xacro:macro name="RobotTrunk" params="name *origin">
 		<!-- Floating-base Joint -->
-		<joint name="${name}_qx_joint" type="revolute">
-			<axis xyz="1 0 0"/>
-			<origin xyz="0 0 0.15" rpy="0 0 0"/>
-			<limit effort="30." velocity="2.0" lower="-0.001" upper="0.001"/>
-			<dynamics damping="0.3" friction="0" />
+		<joint name="${name}_qx_joint" type="fixed">
+			<!-- <axis xyz="1 0 0"/> -->
+			<!-- <origin xyz="0 0 0.0" rpy="0 0 0"/> -->
+			<!-- <limit effort="30." velocity="2.0" lower="-0.001" upper="0.001"/> -->
+			<!-- <dynamics damping="0.3" friction="0" /> -->
 			<parent link="world"/>
 			<child link="trunk"/>
@@ -38,4 +38,5 @@
 		<!-- Extensions -->
 		<xacro:trunk_gazebo name="trunk"/>
+		<!--
 		<transmission name="${name}_qx_trans">
 			<type>transmission_interface/SimpleTransmission</type>
@@ -51,4 +52,5 @@
 			<provideFeedback>true</provideFeedback>
 		</gazebo>
+		-->
 	</xacro:macro>
 </robot>
