Commit message: single leg motion ok;start on controllers

File: corin_description/urdfs/guide_rail/guide_rail.xacro (robot description, xacro)
@@ -42,5 +42,5 @@
 			<axis xyz="0 0 1"/>
 			<origin xyz="0 0 0.0" rpy="0 0 0"/>
-			<limit effort="30." velocity="2.0" lower="-0.02" upper="0.2"/>
+			<limit effort="30." velocity="2.0" lower="-0.02" upper="0.1"/>
 			<dynamics damping="0.5" friction="0" />
 		</joint>

File: corin_description/urdfs/leg/leg.gazebo.xacro (robot description, xacro)
@@ -72,10 +72,11 @@
 		</gazebo>
 		<gazebo reference="${name}_foot">
-			<kp>100000.0</kp>
-			<kd>0.1</kd>
+			<kp>1e5</kp>
+            <kd>10.0</kd>
+            <soft_cfm>0.0</soft_cfm>
+            <soft_erp>0.2</soft_erp>
 			<mu1>1.0</mu1>
 			<mu2>1.0</mu2>
-			<!-- <fdir1>1 0 0</fdir1> -->
-			<maxVel>0.00</maxVel> 		<!-- contact correction velocity truncation -->
+			<maxVel>0.0001</maxVel> 		<!-- contact correction velocity truncation -->
 			<minDepth>0.001</minDepth> 	<!-- penetration between objects -->
 			<material>Gazebo/Black</material>
