Commit message: added snapshot for rviz

File: corin_description/urdfs/common.xacro (robot description, xacro)
@@ -2,4 +2,5 @@
 <robot xmlns:xacro="http://www.ros.org/wiki/xacro" name="corin">
 	<xacro:property name="PI" value="3.1415926535897931"/>
+	<xacro:property name="link_scale" value="1.289"  />
 	<!-- standard distances -->
 	<xacro:property name="trunk_x" value="0.23"/> 		<!-- distance between front & back  joints -->

File: corin_description/urdfs/leg/leg.xacro (robot description, xacro)
@@ -38,5 +38,5 @@
 		<!-- Lower leg joint -->
 		<joint name="${name}_q3_joint" type="revolute">
-			<origin xyz="${femur_l} 0 0" rpy="0 0 0"/>
+			<origin xyz="${femur_l*link_scale} 0 0" rpy="0 0 0"/>
 			<parent link="${name}_upperleg"/>
 			<child  link="${name}_lowerleg"/>
@@ -50,5 +50,5 @@
 		<!-- Foot joint -->
 		<joint name="${name}_foot_joint" type="fixed">
-			<origin xyz="${tibia_l} 0 0" rpy="0 0 0"/>
+			<origin xyz="${tibia_l*link_scale} 0 0" rpy="0 0 0"/>
 			<parent link="${name}_lowerleg"/>
 			<child  link="${name}_foot"/>
@@ -81,5 +81,5 @@
 			<visual>
 		      	<geometry>
-		        	<mesh filename="package://corin_description/meshes/Femur.STL" scale="1 1 1"/>
+		        	<mesh filename="package://corin_description/meshes/Femur.STL" scale="${link_scale} ${link_scale} ${link_scale}"/>
 		      	</geometry>
 		      	<origin xyz="0 0 0" rpy="0 0 0"/>
@@ -103,5 +103,5 @@
 			<visual>
 		      	<geometry>
-		      		<mesh filename="package://corin_description/meshes/Tibia.STL" scale="1 1 1"/>
+		      		<mesh filename="package://corin_description/meshes/Tibia.STL" scale="${link_scale} ${link_scale} ${link_scale}"/>
 		      	</geometry>
 		      	<origin xyz="0 0 0" rpy="${pi/2} 0 0"/>

Commit message: changes to other files

File: corin_description/urdfs/common.xacro (robot description, xacro)
@@ -2,5 +2,5 @@
 <robot xmlns:xacro="http://www.ros.org/wiki/xacro" name="corin">
 	<xacro:property name="PI" value="3.1415926535897931"/>
-	<xacro:property name="link_scale" value="1.289"  />
+	<xacro:property name="link_scale" value="1.067"  /> 	<!-- chimney: 1.267/1.067		wall:1.12  -->
 	<!-- standard distances -->
 	<xacro:property name="trunk_x" value="0.23"/> 		<!-- distance between front & back  joints -->
@@ -58,5 +58,5 @@
 	<xacro:property name="femur_i_zz"  value="0.000051"  />
 	<!--  Tibia assembly -->
-	<xacro:property name="tibia_l" value="0.134" />
+	<xacro:property name="tibia_l" value="0.15" />
 	<xacro:property name="tibia_w" value="0.04" />
 	<xacro:property name="tibia_d" value="0.025" />

File: corin_description/urdfs/leg/leg.xacro (robot description, xacro)
@@ -50,5 +50,5 @@
 		<!-- Foot joint -->
 		<joint name="${name}_foot_joint" type="fixed">
-			<origin xyz="${tibia_l*link_scale} 0 0" rpy="0 0 0"/>
+			<origin xyz="${tibia_l*link_scale-foot_r} 0 0" rpy="0 0 0"/>
 			<parent link="${name}_lowerleg"/>
 			<child  link="${name}_foot"/>
@@ -81,5 +81,5 @@
 			<visual>
 		      	<geometry>
-		        	<mesh filename="package://corin_description/meshes/Femur.STL" scale="${link_scale} ${link_scale} ${link_scale}"/>
+		        	<mesh filename="package://corin_description/meshes/Femur.STL" scale="${link_scale} 1 1"/>
 		      	</geometry>
 		      	<origin xyz="0 0 0" rpy="0 0 0"/>
@@ -103,5 +103,5 @@
 			<visual>
 		      	<geometry>
-		      		<mesh filename="package://corin_description/meshes/Tibia.STL" scale="${link_scale} ${link_scale} ${link_scale}"/>
+		      		<mesh filename="package://corin_description/meshes/Tibia.STL" scale="${link_scale+0.05} 1 1"/>
 		      	</geometry>
 		      	<origin xyz="0 0 0" rpy="${pi/2} 0 0"/>

Commit message: resolving iros demo

File: corin_description/urdfs/common.xacro (robot description, xacro)
@@ -2,5 +2,5 @@
 <robot xmlns:xacro="http://www.ros.org/wiki/xacro" name="corin">
 	<xacro:property name="PI" value="3.1415926535897931"/>
-	<xacro:property name="link_scale" value="1.067"  /> 	<!-- chimney: 1.267/1.067		wall:1.12  -->
+	<xacro:property name="link_scale" value="0.974"  /> 	<!-- chimney: 1.267/1.067		wall:1.12  -->
 	<!-- standard distances -->
 	<xacro:property name="trunk_x" value="0.23"/> 		<!-- distance between front & back  joints -->

Commit message: presentation for rain

File: corin_description/urdfs/common.xacro (robot description, xacro)
@@ -2,5 +2,5 @@
 <robot xmlns:xacro="http://www.ros.org/wiki/xacro" name="corin">
 	<xacro:property name="PI" value="3.1415926535897931"/>
-	<xacro:property name="link_scale" value="0.974"  /> 	<!-- chimney: 1.267/1.067		wall:1.12  -->
+	<xacro:property name="link_scale" value="0.7"  /> 	<!-- chimney: 1.267/1.067		wall:1.12/0.974  -->
 	<!-- standard distances -->
 	<xacro:property name="trunk_x" value="0.23"/> 		<!-- distance between front & back  joints -->

Commit message: updated common.xacro

File: corin_description/urdfs/common.xacro (robot description, xacro)
@@ -2,5 +2,5 @@
 <robot xmlns:xacro="http://www.ros.org/wiki/xacro" name="corin">
 	<xacro:property name="PI" value="3.1415926535897931"/>
-	<xacro:property name="link_scale" value="0.7"  /> 	<!-- chimney: 1.267/1.067		wall:1.12/0.974  -->
+	<xacro:property name="link_scale" value="1.0"  /> 	<!-- chimney: 1.267/1.067		wall:1.12/0.974  -->
 	<!-- standard distances -->
 	<xacro:property name="trunk_x" value="0.23"/> 		<!-- distance between front & back  joints -->

Commit message: setting up new branch

File: corin_description/urdfs/common.xacro (robot description, xacro)
@@ -2,5 +2,5 @@
 <robot xmlns:xacro="http://www.ros.org/wiki/xacro" name="corin">
 	<xacro:property name="PI" value="3.1415926535897931"/>
-	<xacro:property name="link_scale" value="1.0"  /> 	<!-- chimney: 1.267/1.067		wall:1.12/0.974  -->
+	<xacro:property name="link_scale" value="1.267"  /> 	<!-- chimney: 1.267/1.067		wall:1.12/0.974  -->
 	<!-- standard distances -->
 	<xacro:property name="trunk_x" value="0.23"/> 		<!-- distance between front & back  joints -->

Commit message: working on wall cornering

File: corin_description/urdfs/common.xacro (robot description, xacro)
@@ -2,5 +2,5 @@
 <robot xmlns:xacro="http://www.ros.org/wiki/xacro" name="corin">
 	<xacro:property name="PI" value="3.1415926535897931"/>
-	<xacro:property name="link_scale" value="1.267"  /> 	<!-- chimney: 1.267/1.067		wall:1.12/0.974  -->
+	<xacro:property name="link_scale" value="1.333"  /> 	<!-- chimney: 1.267/1.067		wall:1.12/0.974  -->
 	<!-- standard distances -->
 	<xacro:property name="trunk_x" value="0.23"/> 		<!-- distance between front & back  joints -->

Commit message: working on wall

File: corin_description/urdfs/common.xacro (robot description, xacro)
@@ -2,5 +2,6 @@
 <robot xmlns:xacro="http://www.ros.org/wiki/xacro" name="corin">
 	<xacro:property name="PI" value="3.1415926535897931"/>
-	<xacro:property name="link_scale" value="1.333"  /> 	<!-- chimney: 1.267/1.067		wall:1.12/0.974  -->
+	<xacro:property name="link_scale" value="1.0"  /> 	<!-- chimney: 1.267/1.067		wall:1.12/0.974  -->
+ 															<!-- chimney: 1.333 for error margin -->
 	<!-- standard distances -->
 	<xacro:property name="trunk_x" value="0.23"/> 		<!-- distance between front & back  joints -->

Commit message: wall convex corner works

File: corin_description/urdfs/common.xacro (robot description, xacro)
@@ -12,5 +12,5 @@
 	<xacro:property name="MX64_effort"    value="2.85" /> 					<!-- real: 2.85 Nm 	-->
 	<xacro:property name="MX64_velocity"  value="5.23" />
-	<xacro:property name="cox_joint_lim" value="1.00" />	<!-- 57deg -->
+	<xacro:property name="cox_joint_lim" value="1.05" />	<!-- 57deg -->
 	<xacro:property name="cxm_joint_lim" value="0.84" />	<!-- 48deg -->
 	<xacro:property name="fem_joint_lim" value="2.22" />	<!-- 127deg -->

Commit message: stabilipy search direction modified to be robust to small distance between the inner and outer vertex

File: corin_description/urdfs/common.xacro (robot description, xacro)
@@ -36,5 +36,5 @@
 	<xacro:property name="coxa_com_y" value="0"  />
 	<xacro:property name="coxa_com_z" value="0"  />
-	<xacro:property name="coxa_m"     value="0.0406" />
+	<xacro:property name="coxa_m"     value="0.040586"  />
 	<xacro:property name="coxa_i_xx"  value="0.000038"  />
 	<xacro:property name="coxa_i_xy"  value="0.0"  />
@@ -51,6 +51,6 @@
 	<xacro:property name="femur_com_y" value="0"  />
 	<xacro:property name="femur_com_z" value="0"  />
-	<xacro:property name="femur_m"     value="0.35" />
-	<xacro:property name="femur_i_xx"  value="0.000014"  />
+	<xacro:property name="femur_m"     value="0.347529" />
+	<xacro:property name="femur_i_xx"  value="0.000014" />
 	<xacro:property name="femur_i_xy"  value="0"  />
 	<xacro:property name="femur_i_xz"  value="0"  />
@@ -66,5 +66,5 @@
 	<xacro:property name="tibia_com_y" value="0"  		/>
 	<xacro:property name="tibia_com_z" value="0"  		/>
-	<xacro:property name="tibia_m"     value="0.076" 	/>
+	<xacro:property name="tibia_m"     value="0.06313" 	/> 	<!-- 0.076 -->
 	<xacro:property name="tibia_i_xx"  value="0.000025" />
 	<xacro:property name="tibia_i_xy"  value="0"  		/>

Commit message: working on jerk in position control for base tracking

File: corin_description/urdfs/common.xacro (robot description, xacro)
@@ -9,5 +9,5 @@
 	<xacro:property name="trunk_z" value="0.07"/>
 	<!--  Joint parameters -->
-	<xacro:property name="MX64_damping"   value="0.15" /> 					<!-- real: 0.2 		-->
+	<xacro:property name="MX64_damping"   value="0.20" /> 					<!-- real: 0.2 		-->
 	<xacro:property name="MX64_effort"    value="2.85" /> 					<!-- real: 2.85 Nm 	-->
 	<xacro:property name="MX64_velocity"  value="5.23" />

Commit message: resolved gait cycle

File: corin_description/urdfs/common.xacro (robot description, xacro)
@@ -78,3 +78,5 @@
 	<xacro:property name="foot_I" value="0.000004" />
 	<!-- Rectangular box: m*(a^2 + b^2)/12 -->
+	<xacro:property name="light_grey" value="0.8" />
+	<xacro:property name="dark_grey" value="0.1" />
 </robot>

File: corin_description/urdfs/leg/leg.xacro (robot description, xacro)
@@ -62,5 +62,7 @@
 			        <mesh filename="package://corin_description/meshes/Coxa.STL" scale="1 1 1"/>
 			      </geometry>
-		      	<material name="green"/>
+		      	<material name="Green1">
+			       <color rgba="0.06 0.886 0.764 0.7"/>
+			    </material>
 		    </visual>
 		    <collision>
@@ -69,5 +71,5 @@
 			      <mesh filename="package://corin_description/meshes/Coxa_collision.STL" scale="1 1 1"/>
 			    </geometry>
-		      <material name="orange"/>
+		      	<material name="grey"/>
 		    </collision>
 		    <inertial>
@@ -84,5 +86,7 @@
 		      	</geometry>
 		      	<origin xyz="0 0 0" rpy="0 0 0"/>
-		      	<material name="blue"/>
+		      	<material name="LightGrey">
+			       <color rgba="${light_grey} ${light_grey} ${light_grey} 0.7"/>
+			    </material>
 		    </visual>
 		    <collision>
@@ -106,10 +110,11 @@
 		      	</geometry>
 		      	<origin xyz="0 0 0" rpy="${pi/2} 0 0"/>
-		      	<material name="yellow"/>
+		      	<material name="LightGrey">
+			       <color rgba="${light_grey} ${light_grey} ${light_grey} 0.7"/>
+			    </material>
 		    </visual>
 		    <collision>
 		      	<geometry>
-							<mesh filename="package://corin_description/meshes/Tibia_collision.STL" scale="1 1 1"/>
-		        	<!-- <box size= "${tibia_cl} ${tibia_d} ${tibia_w}"/> -->
+					<mesh filename="package://corin_description/meshes/Tibia_collision.STL" scale="1 1 1"/>
 		      	</geometry>
 		      	<origin xyz="0.0 0 0" rpy="${pi/2} 0 0"/>
@@ -129,5 +134,7 @@
 		      	</geometry>
 		      	<origin xyz="0 0 0" rpy="0 0 0"/>
-		      	<material name="black"/>
+		      	<material name="DarkGrey">
+			       <color rgba="${dark_grey} ${dark_grey} ${dark_grey} 0.7"/>
+			    </material>
 		    </visual>
 		    <collision>

File: corin_description/urdfs/trunk/trunk_fixed.xacro (robot description, xacro)
@@ -27,5 +27,7 @@
 					<mesh filename="package://corin_description/meshes/Body.STL" scale="1 1 1"/>
 				</geometry>
-				<material name="orange"/>
+				<material name="MidGrey">
+			       <color rgba="0.5 0.5 0.5 0.7"/>
+			    </material>
 			</visual>
 			<collision>

File: corin_description/urdfs/trunk/trunk_model.xacro (robot description, xacro)
@@ -34,5 +34,7 @@
 					<!-- <box size= "${trunk_x} ${trunk_y} ${trunk_z}"/> -->
 				</geometry>
-				<material name="orange"/>
+				<material name="MidGrey">
+			       <color rgba="0.5 0.5 0.5 0.7"/>
+			    </material>
 			</visual>
 			<collision>

Commit message: added comments for state estimation

File: corin_description/urdfs/common.xacro (robot description, xacro)
@@ -12,6 +12,6 @@
 	<xacro:property name="MX64_effort"    value="2.85" /> 					<!-- real: 2.85 Nm 	-->
 	<xacro:property name="MX64_velocity"  value="5.23" />
-	<xacro:property name="cox_joint_lim" value="1.05" />	<!-- 57deg -->
-	<xacro:property name="cxm_joint_lim" value="0.84" />	<!-- 48deg -->
+	<xacro:property name="cox_joint_lim" value="2.05" />	<!-- 57 deg = 1.05 rad -->
+	<xacro:property name="cxm_joint_lim" value="2.84" />	<!-- 48 deg = 0.84 rad -->
 	<xacro:property name="fem_joint_lim" value="2.22" />	<!-- 127deg -->
 	<xacro:property name="tib_joint_lim" value="2.79" /> 	<!-- 160.5 -->

Commit message: code for testing hardware open-loop stability

File: corin_description/urdfs/common.xacro (robot description, xacro)
@@ -11,5 +11,5 @@
 	<xacro:property name="MX64_damping"   value="0.20" /> 					<!-- real: 0.2 		-->
 	<xacro:property name="MX64_effort"    value="2.85" /> 					<!-- real: 2.85 Nm 	-->
-	<xacro:property name="MX64_velocity"  value="5.23" />
+	<xacro:property name="MX64_velocity"  value="6.6" />
 	<xacro:property name="cox_joint_lim" value="2.05" />	<!-- 57 deg = 1.05 rad -->
 	<xacro:property name="cxm_joint_lim" value="2.84" />	<!-- 48 deg = 0.84 rad -->

File: corin_description/urdfs/leg/leg.gazebo.xacro (robot description, xacro)
@@ -42,6 +42,6 @@
 		</xacro:if>
 		<gazebo reference="${name}_hipassembly">
-			<kp>1000000.0</kp>
-			<kd>100.0</kd>
+			<kp>1e5</kp>
+            <kd>10.0</kd>
 			<mu1>1.5</mu1>
 			<mu2>1.5</mu2>
@@ -52,6 +52,6 @@
 		</gazebo>
 		<gazebo reference="${name}_upperleg">
-			<kp>1000000.0</kp>
-			<kd>100.0</kd>
+			<kp>1e5</kp>
+            <kd>10.0</kd>
 			<mu1>1.5</mu1>
 			<mu2>1.5</mu2>
@@ -62,6 +62,6 @@
 		</gazebo>
 		<gazebo reference="${name}_lowerleg">
-			<kp>1000000.0</kp>
-			<kd>100.0</kd>
+			<kp>1e5</kp>
+            <kd>10.0</kd>
 			<mu1>1.5</mu1>
 			<mu2>1.5</mu2>
@@ -75,7 +75,8 @@
             <kd>10.0</kd>
             <soft_cfm>0.0</soft_cfm>
-            <soft_erp>0.2</soft_erp>
+            <soft_erp>0.01</soft_erp>
 			<mu1>1.0</mu1>
 			<mu2>1.0</mu2>
+			<fdir1>1 0 0</fdir1>
 			<maxVel>0.0001</maxVel> 		<!-- contact correction velocity truncation -->
 			<minDepth>0.001</minDepth> 	<!-- penetration between objects -->

Commit message: Revert "code for testing hardware open-loop stability"
This reverts commit 39bfc0096c5d21967ab3d02bb9f6f0fa2e30b297.

File: corin_description/urdfs/common.xacro (robot description, xacro)
@@ -11,5 +11,5 @@
 	<xacro:property name="MX64_damping"   value="0.20" /> 					<!-- real: 0.2 		-->
 	<xacro:property name="MX64_effort"    value="2.85" /> 					<!-- real: 2.85 Nm 	-->
-	<xacro:property name="MX64_velocity"  value="6.6" />
+	<xacro:property name="MX64_velocity"  value="5.23" />
 	<xacro:property name="cox_joint_lim" value="2.05" />	<!-- 57 deg = 1.05 rad -->
 	<xacro:property name="cxm_joint_lim" value="2.84" />	<!-- 48 deg = 0.84 rad -->

File: corin_description/urdfs/leg/leg.gazebo.xacro (robot description, xacro)
@@ -42,6 +42,6 @@
 		</xacro:if>
 		<gazebo reference="${name}_hipassembly">
-			<kp>1e5</kp>
-            <kd>10.0</kd>
+			<kp>1000000.0</kp>
+			<kd>100.0</kd>
 			<mu1>1.5</mu1>
 			<mu2>1.5</mu2>
@@ -52,6 +52,6 @@
 		</gazebo>
 		<gazebo reference="${name}_upperleg">
-			<kp>1e5</kp>
-            <kd>10.0</kd>
+			<kp>1000000.0</kp>
+			<kd>100.0</kd>
 			<mu1>1.5</mu1>
 			<mu2>1.5</mu2>
@@ -62,6 +62,6 @@
 		</gazebo>
 		<gazebo reference="${name}_lowerleg">
-			<kp>1e5</kp>
-            <kd>10.0</kd>
+			<kp>1000000.0</kp>
+			<kd>100.0</kd>
 			<mu1>1.5</mu1>
 			<mu2>1.5</mu2>
@@ -75,8 +75,7 @@
             <kd>10.0</kd>
             <soft_cfm>0.0</soft_cfm>
-            <soft_erp>0.01</soft_erp>
+            <soft_erp>0.2</soft_erp>
 			<mu1>1.0</mu1>
 			<mu2>1.0</mu2>
-			<fdir1>1 0 0</fdir1>
 			<maxVel>0.0001</maxVel> 		<!-- contact correction velocity truncation -->
 			<minDepth>0.001</minDepth> 	<!-- penetration between objects -->

Commit message: wall corner concave and convex working

File: corin_description/urdfs/common.xacro (robot description, xacro)
@@ -18,5 +18,5 @@
 	<!-- Inertial values -->
 	<!-- Trunk  -->
-	<xacro:property name="xcom_trunk" value="0.0"/>
+	<xacro:property name="xcom_trunk" value="-0.0"/>
 	<xacro:property name="ycom_trunk" value="0.0"/>
 	<xacro:property name="zcom_trunk" value="0.0"/>

Commit message: logged data for chimney nominal

File: corin_description/urdfs/common.xacro (robot description, xacro)
@@ -10,6 +10,6 @@
 	<!--  Joint parameters -->
 	<xacro:property name="MX64_damping"   value="0.20" /> 					<!-- real: 0.2 		-->
-	<xacro:property name="MX64_effort"    value="2.85" /> 					<!-- real: 2.85 Nm 	-->
-	<xacro:property name="MX64_velocity"  value="5.23" />
+	<xacro:property name="MX64_effort"    value="6.0" /> 					<!-- real: 2.85 Nm 	-->
+	<xacro:property name="MX64_velocity"  value="4.0" />
 	<xacro:property name="cox_joint_lim" value="2.05" />	<!-- 57 deg = 1.05 rad -->
 	<xacro:property name="cxm_joint_lim" value="2.84" />	<!-- 48 deg = 0.84 rad -->
@@ -77,4 +77,5 @@
 	<xacro:property name="foot_m" value="0.040"   />
 	<xacro:property name="foot_I" value="0.000004" />
+	<xacro:property name="foot_friction" value="0.5" />
 	<!-- Rectangular box: m*(a^2 + b^2)/12 -->
 	<xacro:property name="light_grey" value="0.8" />

File: corin_description/urdfs/leg/leg.gazebo.xacro (robot description, xacro)
@@ -76,6 +76,6 @@
             <soft_cfm>0.0</soft_cfm>
             <soft_erp>0.2</soft_erp>
-			<mu1>1.0</mu1>
-			<mu2>1.0</mu2>
+			<mu1>${foot_friction}</mu1>
+			<mu2>${foot_friction}</mu2>
 			<maxVel>0.0001</maxVel> 		<!-- contact correction velocity truncation -->
 			<minDepth>0.001</minDepth> 	<!-- penetration between objects -->

Commit message: added funcationality for robot to wall walk smooth

File: corin_description/urdfs/common.xacro (robot description, xacro)
@@ -77,5 +77,5 @@
 	<xacro:property name="foot_m" value="0.040"   />
 	<xacro:property name="foot_I" value="0.000004" />
-	<xacro:property name="foot_friction" value="0.5" />
+	<xacro:property name="foot_friction" value="1.0" />
 	<!-- Rectangular box: m*(a^2 + b^2)/12 -->
 	<xacro:property name="light_grey" value="0.8" />
