Commit message: robot can be kinematically simulated using only rviz; gait_class update functions improved

File: corin_description/urdfs/leg/leg.xacro (robot description, xacro)
@@ -129,5 +129,5 @@
 		      	</geometry>
 		      	<origin xyz="0 0 0" rpy="0 0 0"/>
-		      	<material name="blue"/>
+		      	<material name="black"/>
 		    </visual>
 		    <collision>

Commit message: making chimney walking work

File: corin_description/urdfs/leg/leg.xacro (robot description, xacro)
@@ -116,5 +116,5 @@
 		    <collision>
 		      	<geometry>
-					<mesh filename="package://corin_description/meshes/Tibia_collision.STL" scale="1 1 1"/>
+					<mesh filename="package://corin_description/meshes/Tibia_collision.STL" scale="0.1 0.1 0.1"/>
 		      	</geometry>
 		      	<origin xyz="0.0 0 0" rpy="${pi/2} 0 0"/>

Commit message: robot_validation chimney walking data collected (analysis required)

File: corin_description/urdfs/leg/leg.xacro (robot description, xacro)
@@ -116,5 +116,6 @@
 		    <collision>
 		      	<geometry>
-					<mesh filename="package://corin_description/meshes/Tibia_collision.STL" scale="0.1 0.1 0.1"/>
+					<!-- <mesh filename="package://corin_description/meshes/Tibia.STL" scale="${link_scale+0.05} 1 1"/> -->
+					<mesh filename="package://corin_description/meshes/Tibia.STL" scale="0.1 0.1 0.1"/>
 		      	</geometry>
 		      	<origin xyz="0.0 0 0" rpy="${pi/2} 0 0"/>

File: corin_description/urdfs/sensors/sensors.xacro (robot description, xacro)
@@ -19,5 +19,5 @@
                 <origin xyz="0.0 0 0.0" rpy="0 0 0"/>
                 <geometry>
-                    <box size="0.05 0.05 0.01" />
+                    <box size="0.001 0.001 0.001" />
                 </geometry>
                 <material name="black">
@@ -27,5 +27,5 @@
         </link>
         <gazebo>
-            <material>Gazebo/Red</material>
+            <material>Gazebo/DarkGrey</material>
             <plugin name="imu_plugin" filename="libgazebo_ros_imu.so">
                 <robotNamespace>/corin/imu/</robotNamespace>

File: corin_description/urdfs/trunk/trunk_model.xacro (robot description, xacro)
@@ -17,5 +17,5 @@
 			<visual>
 				<geometry>
-					<cylinder length="0.01" radius="0.01"/>
+					<cylinder length="0.001" radius="0.001"/>
 				</geometry>
 			</visual>

Commit message: robot_validation chimney walking data collected (new n correct)

File: corin_description/urdfs/leg/leg.xacro (robot description, xacro)
@@ -116,6 +116,6 @@
 		    <collision>
 		      	<geometry>
-					<!-- <mesh filename="package://corin_description/meshes/Tibia.STL" scale="${link_scale+0.05} 1 1"/> -->
-					<mesh filename="package://corin_description/meshes/Tibia.STL" scale="0.1 0.1 0.1"/>
+					<mesh filename="package://corin_description/meshes/Tibia.STL" scale="${link_scale+0.05} 1 1"/>
+					<!-- <mesh filename="package://corin_description/meshes/Tibia.STL" scale="0.1 0.1 0.1"/> -->
 		      	</geometry>
 		      	<origin xyz="0.0 0 0" rpy="${pi/2} 0 0"/>

Commit message: chimney cornering now imports surface normal; issue with contact force for cornering

File: corin_description/urdfs/leg/leg.xacro (robot description, xacro)
@@ -51,4 +51,5 @@
 		<joint name="${name}_foot_joint" type="fixed">
 			<origin xyz="${tibia_l*link_scale-foot_r} 0 0" rpy="0 0 0"/>
+			<!-- <origin xyz="${tibia_l*link_scale} 0 0" rpy="0 0 0"/> -->
 			<parent link="${name}_lowerleg"/>
 			<child  link="${name}_foot"/>

Commit message: Evaluated wall CONVEX  corner for base control

File: corin_description/urdfs/leg/leg.xacro (robot description, xacro)
@@ -116,5 +116,6 @@
 		    <collision>
 		      	<geometry>
-					<mesh filename="package://corin_description/meshes/Tibia_collision.STL" scale="0.1 0.1 0.1"/>
+					<!-- <mesh filename="package://corin_description/meshes/Tibia_collision.STL" scale="0.1 0.1 0.1"/> -->
+					<mesh filename="package://corin_description/meshes/Tibia.STL" scale="${link_scale+0.05} 1 1"/>
 		      	</geometry>
 		      	<origin xyz="0.0 0 0" rpy="${pi/2} 0 0"/>

Commit message: gazebo evaluation of chimney nominal

File: corin_description/urdfs/leg/leg.xacro (robot description, xacro)
@@ -117,6 +117,6 @@
 		    <collision>
 		      	<geometry>
-					<mesh filename="package://corin_description/meshes/Tibia.STL" scale="${link_scale+0.05} 1 1"/>
-					<!-- <mesh filename="package://corin_description/meshes/Tibia.STL" scale="0.1 0.1 0.1"/> -->
+					<!-- <mesh filename="package://corin_description/meshes/Tibia.STL" scale="${link_scale+0.05} 1 1"/> -->
+					<mesh filename="package://corin_description/meshes/Tibia.STL" scale="0.1 0.1 0.1"/>
 		      	</geometry>
 		      	<origin xyz="0.0 0 0" rpy="${pi/2} 0 0"/>

Commit message: gazebo chimney nominal data collected

File: corin_description/urdfs/leg/leg.xacro (robot description, xacro)
@@ -117,5 +117,5 @@
 		    <collision>
 		      	<geometry>
-					<!-- <mesh filename="package://corin_description/meshes/Tibia.STL" scale="${link_scale+0.05} 1 1"/> -->
+					<!--<mesh filename="package://corin_description/meshes/Tibia.STL" scale="${link_scale+0.05} 1 1"/> -->
 					<mesh filename="package://corin_description/meshes/Tibia.STL" scale="0.1 0.1 0.1"/>
 		      	</geometry>

Commit message: evaluated gazebo simulation of chimney and wall transition

File: corin_description/urdfs/leg/leg.xacro (robot description, xacro)
@@ -94,4 +94,5 @@
 		      	<geometry>
 		        	<box size= "${femur_cl} ${femur_w} ${femur_d}"/>
+		        	<!-- <box size= "0.01 0.01 0.01"/> -->
 		      	</geometry>
 		      	<origin xyz="0.075 0 0" rpy="0 0 0"/>
