Commit message: Code cleanup for simple demo -walkleft and walkright tested for 0.5m distance each

File: corin_description/urdfs/sensors/sensors.xacro (robot description, xacro)
@@ -19,5 +19,5 @@
                 <origin xyz="0.0 0 0.0" rpy="0 0 0"/>
                 <geometry>
-                    <box size="0.05 0.1 0.01" />
+                    <box size="0.01 0.01 0.01" />
                 </geometry>
                 <material name="black">
@@ -28,5 +28,5 @@
 								<origin xyz="0.0 0 0.0" rpy="0 0 0"/>
 								<geometry>
-										<box size="0.05 0.1 0.01" />
+										<box size="0.01 0.01 0.01" />
 								</geometry>
 								<material name="black">
@@ -36,5 +36,5 @@
         </link>
         <gazebo reference="${imu_name}">
-					<material>Gazebo/Red</material>
+					<material>Gazebo/Grey</material>
 					<gravity>false</gravity>
 					<sensor name='IMU' type='imu'>
